File: hardware/HUBCHIP.kicad_sch (KiCad schematic)
At the start: 36 parts, among them Y1 25MHz

Commit message: finnished rudimentry schimatics still needs alot of work
Parts:
- removed JP1: HOST_TYPE0, symbol Jumper:SolderJumper_3_Bridged12
- removed JP2: HOST_TYPE1, symbol Jumper:SolderJumper_3_Bridged12
- added JP5 (x4): ~, symbol Jumper:SolderJumper_3_Open
Connections:
- net +3V3: now also JP5.1 (A), JP5.1 (A), JP5.1 (A), JP5.1 (A)
- net GND: now also JP5.3 (B), JP5.3 (B), JP5.3 (B), JP5.3 (B); no longer U12.61 (CC_POL/GPIO71), U12.63 (ALT_MUX_EN/GPIO70)
- net at U12.53 (HOST_TYPE0/GPIO23): now also JP5.2 (C)
- net at U12.55 (HOST_TYPE1/GPIO67): now also JP5.2 (C)
- new net: JP5.2 (C), U12.61 (CC_POL/GPIO71)
- new net: JP5.2 (C), U12.63 (ALT_MUX_EN/GPIO70)
Other:
- note added: "ALL SHOLD BE PULLED DOWN"

Commit message: working on hardware
Parts:
- added J1: ~, symbol Connector:Conn_01x01_Pin
- added JP4: ~, Jumper:SolderJumper-3_P1.3mm_Open_RoundedPad1.0x1.5mm_NumberLabels, symbol Jumper:SolderJumper_3_Open
- added R79: 10K, symbol Device:R
- added TP1: TestPoint, TestPoint:TestPoint_Pad_D1.0mm, symbol Connector:TestPoint
- C53: renamed from C57; footprint (none) -> Capacitor_SMD:C_0603_1608Metric
- C54: renamed from C58; footprint (none) -> Capacitor_SMD:C_0603_1608Metric
- C55: renamed from C56; footprint (none) -> Capacitor_SMD:C_0603_1608Metric
- C56: renamed from C52; footprint (none) -> Capacitor_SMD:C_0603_1608Metric
- C57: renamed from C73; value C -> 18pF; footprint (none) -> Capacitor_SMD:C_0603_1608Metric
- C58: renamed from C74; value C -> 18Pf; footprint (none) -> Capacitor_SMD:C_0603_1608Metric
- C59: renamed from C55; footprint (none) -> Capacitor_SMD:C_0603_1608Metric
- C60: renamed from C49; footprint (none) -> Capacitor_SMD:C_0603_1608Metric
- C61: renamed from C54; footprint (none) -> Capacitor_SMD:C_0603_1608Metric
- C62: renamed from C50; footprint (none) -> Capacitor_SMD:C_0603_1608Metric
- C63: renamed from C53; footprint (none) -> Capacitor_SMD:C_0603_1608Metric
- C64: renamed from C51; footprint (none) -> Capacitor_SMD:C_0603_1608Metric
- C65: renamed from C66; footprint (none) -> Capacitor_SMD:C_0603_1608Metric
- C66: renamed from C65; footprint (none) -> Capacitor_SMD:C_0603_1608Metric
- C67: renamed from C64; footprint (none) -> Capacitor_SMD:C_0603_1608Metric
- C68: renamed from C63; footprint (none) -> Capacitor_SMD:C_0603_1608Metric
- C69: renamed from C62; footprint (none) -> Capacitor_SMD:C_0603_1608Metric
- C70: renamed from C61; footprint (none) -> Capacitor_SMD:C_0603_1608Metric
- C71: renamed from C60; footprint (none) -> Capacitor_SMD:C_0603_1608Metric
- C72: renamed from C59; footprint (none) -> Capacitor_SMD:C_0603_1608Metric
- C73: renamed from C67; footprint (none) -> Capacitor_SMD:C_0603_1608Metric
- C74: renamed from C68; footprint (none) -> Capacitor_SMD:C_0603_1608Metric
- C75: renamed from C70; footprint (none) -> Capacitor_SMD:C_0603_1608Metric
- C76: renamed from C69; footprint (none) -> Capacitor_SMD:C_0603_1608Metric
- C77: renamed from C72; footprint (none) -> Capacitor_SMD:C_0603_1608Metric
- C78: renamed from C71; footprint (none) -> Capacitor_SMD:C_0603_1608Metric
- JP5: footprint (none) -> Jumper:SolderJumper-3_P1.3mm_Open_RoundedPad1.0x1.5mm_NumberLabels
- Y1: footprint (none) -> Crystal:Crystal_SMD_HC49-SD
- renumbered R79 to R80, R80 to R81, R81 to R82, R78 to R83, R76 to R84, R77 to R85, U12 to U13
Connections:
- net +3V3: now also R79.2
- net at U13.25 (RESET_N): now also JP4.2 (C)
- new net: J1.1 (Pin_1), JP4.1 (A), R79.1, TP1.1
- new net RST: JP4.3 (B)
Other:
- note added: "HUB CHIP COMS"
- note added: "HUB CHIP CONFIG"
- note added: "HUB CHIP POWER INPUT"
- moved on the sheet: C53, C54, C55, C56, C57, C58, C59, C60, C61, C62, C63, C64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

Commit message: working assighning footprints still
Parts:
- R79, R80, R81, R82, R83, R84, R85: footprint (none) -> Resistor_SMD:R_0603_1608Metric
Changed lines of the file:
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@@
       (effects (font (size 1.27 1.27)))
     )
-    (property "Footprint" "" (at 198.12 118.618 90)
+    (property "Footprint" "Resistor_SMD:R_0603_1608Metric" (at 198.12 118.618 90)
       (effects (font (size 1.27 1.27)) hide)
     )
@@
       (effects (font (size 1.27 1.27)))
     )
-    (property "Footprint" "" (at 110.49 117.348 90)
+    (property "Footprint" "Resistor_SMD:R_0603_1608Metric" (at 110.49 117.348 90)
       (effects (font (size 1.27 1.27)) hide)
     )
@@
       (effects (font (size 1.27 1.27)))
     )
-    (property "Footprint" "" (at 104.14 141.478 90)
+    (property "Footprint" "Resistor_SMD:R_0603_1608Metric" (at 104.14 141.478 90)
       (effects (font (size 1.27 1.27)) hide)
     )
@@
       (effects (font (size 1.27 1.27)))
     )
-    (property "Footprint" "" (at 104.14 149.098 90)
+    (property "Footprint" "Resistor_SMD:R_0603_1608Metric" (at 104.14 149.098 90)
       (effects (font (size 1.27 1.27)) hide)
     )
@@
       (effects (font (size 1.27 1.27)))
     )
-    (property "Footprint" "" (at 113.03 141.478 90)
+    (property "Footprint" "Resistor_SMD:R_0603_1608Metric" (at 113.03 141.478 90)
       (effects (font (size 1.27 1.27)) hide)
     )
@@
       (effects (font (size 1.27 1.27)))
     )
-    (property "Footprint" "" (at 66.04 117.348 90)
+    (property "Footprint" "Resistor_SMD:R_0603_1608Metric" (at 66.04 117.348 90)
       (effects (font (size 1.27 1.27)) hide)
     )
@@
       (effects (font (size 1.27 1.27)))
     )
-    (property "Footprint" "" (at 189.23 118.618 90)
-      (effects (font (size 1.27 1.27)) hide)
-    )
+    (property "Footprint" "Resistor_SMD:R_0603_1608Metric" (at 189.23 118.618 90)
+      (effects (font (size 1.27 1.27)) hide)
+    )

Commit message: FINALY starting the pcb
Parts:
- J1: footprint (none) -> Connector_PinHeader_2.54mm:PinHeader_1x01_P2.54mm_Vertical
- U13: footprint (none) -> CARTHING:VQFN100_KD_MCH
Changed lines of the file:
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@@
       (effects (font (size 1.27 1.27)) (justify right))
     )
-    (property "Footprint" "" (at 58.42 124.46 0)
+    (property "Footprint" "Connector_PinHeader_2.54mm:PinHeader_1x01_P2.54mm_Vertical" (at 58.42 124.46 0)
       (effects (font (size 1.27 1.27)) hide)
     )
@@
       (effects (font (size 1.27 1.27)))
     )
-    (property "Footprint" "" (at 148.59 115.57 0)
+    (property "Footprint" "CARTHING:VQFN100_KD_MCH" (at 148.59 115.57 0)
       (effects (font (size 1.27 1.27)) hide)
     )
@@
       (effects (font (size 1.27 1.27)))
     )
-    (property "Footprint" "" (at 146.05 5.08 0)
+    (property "Footprint" "CARTHING:VQFN100_KD_MCH" (at 146.05 5.08 0)
       (effects (font (size 1.27 1.27)) hide)
     )
@@
       (effects (font (size 1.27 1.27)))
     )
-    (property "Footprint" "" (at 144.78 72.39 0)
-      (effects (font (size 1.27 1.27)) hide)
-    )
+    (property "Footprint" "CARTHING:VQFN100_KD_MCH" (at 144.78 72.39 0)
+      (effects (font (size 1.27 1.27)) hide)
+    )
