File: hardware/HUBCHIP.kicad_sch (KiCad schematic)
At the start: 42 parts, among them Y1 25MHz

Commit message: working in final routing
Connections:
- net GND: now also U13.101 (VSS/GND); no longer U13.EP (VSS/GND)
- net I2C_SDA: now also U13.74 (SMBDATA/GPIO6/SDA); no longer U13.47 (SMBDATA/GPIO6/SDA)
- no-connect marks 1 -> 3

Commit message: finaliseing pcb layout will come back later for a fresh look
Other:
- company: (none) -> MICK MAKE
- title: (none) -> 200W USB PD 3.1 HUB
Changed lines of the file:
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@@
 (kicad_sch (version 20230121) (generator eeschema)
   (paper "A4")
+  (title_block
+    (title "200W USB PD 3.1 HUB")
+    (date "2023-10-03")
+    (rev "A")
+    (company "MICK MAKE")
+    (comment 1 "THIS IS A 2X 100W USB PD SOURCE ")
+    (comment 2 "HUB USB SPEC 3.1")
+    (comment 3 "TOTAL SYSTEM POWER IS ~275w")
+  )
   (junction (at 132.08 35.56) (diameter 0) (color 0 0 0 0)
   )
