File: hardware/5V USB-A AND MCU POWER.kicad_sch (KiCad schematic)
At the start: 28 parts, among them U2 NCP177BMX330TCG, U3 NCP177BMX330TCG, U4 LMR14050-Q1, U5 NCP177AMX120TCG, U6 NCP177AMX120TCG

Commit message: working assighning footprints still
Parts:
- added TP6, TP7: TestPoint, TestPoint:TestPoint_Pad_D1.0mm, symbol Connector:TestPoint
- R11: value 500R -> 10K; footprint (none) -> Resistor_SMD:R_0603_1608Metric
- R12, R13, R14, R15: footprint (none) -> Resistor_SMD:R_0603_1608Metric
- R9: footprint (none) -> Resistor_SMD:R_2512_6332Metric
Connections:
- net +1V2: now also TP7.1
- net +3V3: now also TP6.1
Changed lines of the file:
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@@
   (junction (at 85.09 34.29) (diameter 0) (color 0 0 0 0)
   )
+  (junction (at 71.12 121.92) (diameter 0) (color 0 0 0 0)
+  )
   (junction (at 66.04 157.48) (diameter 0) (color 0 0 0 0)
   )
@@
   (junction (at 137.16 176.53) (diameter 0) (color 0 0 0 0)
   )
+  (junction (at 151.13 121.92) (diameter 0) (color 0 0 0 0)
+  )
   (junction (at 135.89 176.53) (diameter 0) (color 0 0 0 0)
   )
@@
     (stroke (width 0) (type default))
   )
+  (wire (pts (xy 71.12 121.92) (xy 77.47 121.92))
+    (stroke (width 0) (type default))
+  )
   (wire (pts (xy 78.74 50.8) (xy 77.47 50.8))
     (stroke (width 0) (type default))
@@
     (stroke (width 0) (type default))
   )
-  (wire (pts (xy 66.04 121.92) (xy 77.47 121.92))
+  (wire (pts (xy 66.04 121.92) (xy 71.12 121.92))
     (stroke (width 0) (type default))
   )
@@
     (stroke (width 0) (type default))
   )
+  (wire (pts (xy 151.13 121.92) (xy 157.48 121.92))
+    (stroke (width 0) (type default))
+  )
   (wire (pts (xy 49.53 68.58) (xy 49.53 69.85))
     (stroke (width 0) (type default))
@@
     (stroke (width 0) (type default))
   )
-  (wire (pts (xy 146.05 121.92) (xy 157.48 121.92))
+  (wire (pts (xy 146.05 121.92) (xy 151.13 121.92))
     (stroke (width 0) (type default))
   )
@@
       (effects (font (size 1.27 1.27)) (justify left))
     )
-    (property "Footprint" "" (at 47.752 73.66 90)
+    (property "Footprint" "Resistor_SMD:R_0603_1608Metric" (at 47.752 73.66 90)
       (effects (font (size 1.27 1.27)) hide)
     )
@@
       (effects (font (size 1.27 1.27)) (justify left))
     )
-    (property "Value" "500R" (at 43.688 48.2673 0)
-      (effects (font (size 1.27 1.27)) (justify left))
-    )
-    (property "Footprint" "" (at 40.132 46.99 90)
+    (property "Value" "10K" (at 43.688 48.2673 0)
+      (effects (font (size 1.27 1.27)) (justify left))
+    )
+    (property "Footprint" "Resistor_SMD:R_0603_1608Metric" (at 40.132 46.99 90)
       (effects (font (size 1.27 1.27)) hide)
     )
@@
       (effects (font (size 1.27 1.27)))
     )
-    (property "Footprint" "" (at 100.33 90.678 90)
+    (property "Footprint" "Resistor_SMD:R_0603_1608Metric" (at 100.33 90.678 90)
       (effects (font (size 1.27 1.27)) hide)
     )
@@
     )
   )
+  (symbol (lib_id "Connector:TestPoint") (at 71.12 121.92 0) (unit 1)
+    (in_bom yes) (on_board yes) (dnp no) (fields_autoplaced)
+    (property "Reference" "TP6" (at 72.517 117.9743 0)
+      (effects (font (size 1.27 1.27)) (justify left))
+    )
+    (property "Value" "TestPoint" (at 72.517 119.8953 0)
+      (effects (font (size 1.27 1.27)) (justify left))
+    )
+    (property "Footprint" "TestPoint:TestPoint_Pad_D1.0mm" (at 76.2 121.92 0)
+      (effects (font (size 1.27 1.27)) hide)
+    )
+    (property "Datasheet" "~" (at 76.2 121.92 0)
+      (effects (font (size 1.27 1.27)) hide)
+    )
+    (pin "1")
+    (instances
+      (project "usbc-car-module"
+        (path "/fae025e9-99c5-40c1-af6f-99dc1edbfa43/babd34fb-a18a-4bce-9735-4ab8ec7cd7ca"
+          (reference "TP6") (unit 1)
+        )
+      )
+    )
+  )
   (symbol (lib_id "Device:R") (at 88.9 88.9 90) (unit 1)
     (in_bom yes) (on_board yes) (dnp no) (fields_autoplaced)
@@
       (effects (font (size 1.27 1.27)))
     )
-    (property "Footprint" "" (at 88.9 90.678 90)
+    (property "Footprint" "Resistor_SMD:R_0603_1608Metric" (at 88.9 90.678 90)
       (effects (font (size 1.27 1.27)) hide)
     )
@@
         (path "/fae025e9-99c5-40c1-af6f-99dc1edbfa43/babd34fb-a18a-4bce-9735-4ab8ec7cd7ca"
           (reference "C10") (unit 1)
+        )
+      )
+    )
+  )
+  (symbol (lib_id "Connector:TestPoint") (at 151.13 121.92 0) (unit 1)
+    (in_bom yes) (on_board yes) (dnp no) (fields_autoplaced)
+    (property "Reference" "TP7" (at 152.527 117.9743 0)
+      (effects (font (size 1.27 1.27)) (justify left))
+    )
+    (property "Value" "TestPoint" (at 152.527 119.8953 0)
+      (effects (font (size 1.27 1.27)) (justify left))
+    )
+    (property "Footprint" "TestPoint:TestPoint_Pad_D1.0mm" (at 156.21 121.92 0)
+      (effects (font (size 1.27 1.27)) hide)
+    )
+    (property "Datasheet" "~" (at 156.21 121.92 0)
+      (effects (font (size 1.27 1.27)) hide)
+    )
+    (pin "1")
+    (instances
+      (project "usbc-car-module"
+        (path "/fae025e9-99c5-40c1-af6f-99dc1edbfa43/babd34fb-a18a-4bce-9735-4ab8ec7cd7ca"
+          (reference "TP7") (unit 1)
         )
       )
@@
       (effects (font (size 1.27 1.27)) (justify left))
     )
-    (property "Footprint" "" (at 47.752 83.82 90)
+    (property "Footprint" "Resistor_SMD:R_0603_1608Metric" (at 47.752 83.82 90)
       (effects (font (size 1.27 1.27)) hide)
     )
@@
       (effects (font (size 1.27 1.27)))
     )
-    (property "Footprint" "" (at 144.78 70.358 90)
-      (effects (font (size 1.27 1.27)) hide)
-    )
+    (property "Footprint" "Resistor_SMD:R_2512_6332Metric" (at 144.78 70.358 90)
+      (effects (font (size 1.27 1.27)) hide)
+    )

Commit message: FINALY starting the pcb
Parts:
- U4: footprint (none) -> CARTHING:LMR14050
Changed lines of the file:
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@@
       (effects (font (size 1.27 1.27)))
     )
-    (property "Footprint" "" (at 85.09 48.26 0)
+    (property "Footprint" "CARTHING:LMR14050" (at 85.09 48.26 0)
       (effects (font (size 1.27 1.27)) hide)
     )

Commit message: coldent sleep so came back and did somre routing
Parts:
- added C113, C114: 1uF, Capacitor_SMD:C_0603_1608Metric, symbol Device:C
- added R6: 1K, PCM_Potentiometer_SMD_AKL:Potentiometer_Bourns_TC33X_Vertical, symbol Device:R_Trim
- added U19: NCP177BMX330TCG, CARTHING:VREG_NCP170AMX300TCG, symbol CARTHING:NCP177BMX330TCG-Regulator_Linear
- L2: footprint (none) -> CARTHING:IND25X25CZ
Connections:
- net +3V3: now also C114.1, U19.1 (OUT)
- net +5V: now also C113.1, U19.3 (EN), U19.4 (IN)
- net GND: now also U2.5 (EP), U3.5 (EP), U4.11 (EP), U5.5 (EP), U6.5 (EP), C113.2, C114.2, R6.2, U19.2 (GND), U19.5 (EP); no longer R14.1
- new net: R14.1, R6.1
Other:
- moved on the sheet: C10, C11, C14, C15, C19, C20, C22, C23, R14, TP6, TP7

Commit message: finaliseing pcb layout will come back later for a fresh look
Other:
- company: (none) -> MICK MAKE
- title: (none) -> 200W USB PD 3.1 HUB
Changed lines of the file:
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@@
 (kicad_sch (version 20230121) (generator eeschema)
   (paper "A4")
+  (title_block
+    (title "200W USB PD 3.1 HUB")
+    (date "2023-10-03")
+    (rev "A")
+    (company "MICK MAKE")
+    (comment 1 "THIS IS A 2X 100W USB PD SOURCE ")
+    (comment 2 "HUB USB SPEC 3.1")
+    (comment 3 "TOTAL SYSTEM POWER IS ~275w")
+  )
   (junction (at 95.25 88.9) (diameter 0) (color 0 0 0 0)
   )
