File: hardware/usbc-car-module.kicad_pcb (KiCad board)
At the start: 4 copper layers, 343 parts, among them J10 PROG_PORT, J3 0483930003, J4 0483930003, J5 0483930003, J6 0483930003, J7 USB4200-03-A (VIRT FLAG MOUNT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, J8 USB4200-03-A (VIRT FLAG MOUNT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, J9 684M7W2103L461, Q1 NMOS, Q10 NMOS, Q11 NMOS, Q12 NMOS, Q13 NMOS, Q14 NMOS, Q15 NMOS, Q16 NMOS, Q17 BC847BS-7-F, Q18 PMOS, Q19 PMOS, Q2 NMOS, Q20 PMOS, Q21 PMOS, Q22 PMOS, Q23 PMOS, Q24 PMOS, Q25 PMOS, Q26 NMOS, Q27 AON7421, Q3 PMPB11EN,115, Q4 PMPB11EN,115, Q5 PMPB11EN,115, Q6 PMPB11EN,115, Q7 NMOS, Q8 NMOS, Q9 NMOS, SW1 SW_Push, SW2 SW_Push, SW3 SW_Push, U1 LM51231-Q1, U10 ESP-12F, U11 MCP2558FD-xMF, U14 CP2102N-QFN20, U17 AS1115-BSST, U18 LTC-5723HR, U2 NCP177BMX330TCG, U3 NCP177BMX330TCG, U4 LMR14050-Q1, U5 NCP177AMX120TCG, U6 NCP177AMX120TCG, U8 PI4IOE5V6416LEX, U9 PI4IOE5V6416LEX, Y1 25MHz

Commit message: coldent sleep so came back and did somre routing
Parts:
- added C113: 1uF, Capacitor_SMD:C_0603_1608Metric, F.Cu at (381.6, 88.5)
- added C114: 1uF, Capacitor_SMD:C_0603_1608Metric, F.Cu at (373.4, 85.1)
- added L2: 1.2uH CR75NP-1R2MC, CARTHING:IND25X25CZ, F.Cu at (366.2, 99.2)
- added R106: 1K, PCM_Potentiometer_SMD_AKL:Potentiometer_Bourns_TC33X_Vertical, F.Cu at (364.2, 114.0)
- added U19: NCP177BMX330TCG, CARTHING:VREG_NCP170AMX300TCG, F.Cu at (376.9, 88.4)
- R30: footprint Resistor_SMD:R_0603_1608Metric -> Potentiometer_SMD:Potentiometer_Bourns_TC33X_Vertical
- moved Q11 373.3 mm to (383.0, 36.8), turned to 90 degrees
- moved Q10 368.5 mm to (379.0, 36.8), turned to 90 degrees
- moved R30 366.3 mm to (382.5, 40.7), turned to 90 degrees
- moved Q9 363.8 mm to (375.0, 36.8), turned to 90 degrees
- moved R28 360.4 mm to (379.3, 46.7), turned to -90 degrees
- moved R29 359.4 mm to (377.6, 46.7), turned to 90 degrees
- moved R31 359.1 mm to (376.0, 46.7), turned to 90 degrees
- moved Q7 358.3 mm to (371.0, 36.8), turned to 90 degrees
- moved R33 358.1 mm to (374.3, 46.7), turned to 90 degrees
- moved R32 356.8 mm to (378.5, 40.7), turned to 90 degrees
- moved Q8 355.2 mm to (367.0, 36.8), turned to 90 degrees
- moved R34 354.0 mm to (374.5, 40.7), turned to 90 degrees
- moved R36 351.3 mm to (370.5, 40.7), turned to 90 degrees
- moved R35 350.1 mm to (372.7, 46.7), turned to 90 degrees
- moved L3 349.2 mm to (372.9, 55.2), turned to 180 degrees
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Connections:
- C29 pad 1: Net-(Q3-S) -> Net-(U7-SW1)
- C34 pad 2: Net-(Q5-S) -> Net-(U7-SW2)
- L3 pad 2: Net-(Q3-S) -> Net-(U7-SW1)
- L4 pad 1: Net-(Q5-S) -> Net-(U7-SW2)
- Q10 pad 2: F_USB-C_BUCK_9V_SEL -> F_USB-C_BUCK_15V_SEL
- Q11 pad 2: F_USB-C_BUCK_5V_SEL -> F_USB-C_BUCK_20V_SEL
- Q12 pad 2: B_USB-C_BUCK_20V_SEL -> B_USB-C_BUCK_5V_SEL
- Q13 pad 2: B_USB-C_BUCK_15V_SEL -> B_USB-C_BUCK_9V_SEL
- Q15 pad 2: B_USB-C_BUCK_9V_SEL -> B_USB-C_BUCK_15V_SEL
- Q16 pad 2: B_USB-C_BUCK_5V_SEL -> B_USB-C_BUCK_20V_SEL
- Q3 pad 1: Net-(Q3-G) -> +21V
- Q3 pad 3: Net-(Q3-S) -> Net-(Q3-G)
- Q3 pad 4: (no net) -> Net-(U7-SW1)
- Q3 pad 5: (no net) -> +21V
- Q3 pad 6: (no net) -> +21V
- Q3 pad 7: (no net) -> +21V
- Q3 pad 8: (no net) -> Net-(U7-SW1)
- Q4 pad 1: Net-(Q4-G) -> Net-(U7-SW1)
- Q4 pad 2: Net-(Q3-S) -> Net-(U7-SW1)
- Q4 pad 3: GND -> Net-(Q4-G)
- Q4 pad 4: (no net) -> GND
- Q4 pad 5: (no net) -> Net-(U7-SW1)
- Q4 pad 6: (no net) -> Net-(U7-SW1)
- Q4 pad 7: (no net) -> Net-(U7-SW1)
- Q4 pad 8: (no net) -> GND
- Q5 pad 1: Net-(Q5-G) -> +21V
- Q5 pad 3: Net-(Q5-S) -> Net-(Q5-G)
- Q5 pad 4: (no net) -> Net-(U7-SW2)
- Q5 pad 5: (no net) -> +21V
- Q5 pad 6: (no net) -> +21V
- Q5 pad 7: (no net) -> +21V
- Q5 pad 8: (no net) -> Net-(U7-SW2)
- Q6 pad 1: Net-(Q6-G) -> Net-(U7-SW2)
- Q6 pad 2: Net-(Q5-S) -> Net-(U7-SW2)
- Q6 pad 3: GND -> Net-(Q6-G)
- Q6 pad 4: (no net) -> GND
- Q6 pad 5: (no net) -> Net-(U7-SW2)
- Q6 pad 6: (no net) -> Net-(U7-SW2)
- Q6 pad 7: (no net) -> Net-(U7-SW2)
- Q6 pad 8: (no net) -> GND
- Q7 pad 2: F_USB-C_BUCK_20V_SEL -> F_USB-C_BUCK_9V_SEL
- Q8 pad 2: F_USB-C_BUCK_15V_SEL -> F_USB-C_BUCK_5V_SEL
- R14 pad 1: GND -> Net-(R106-Pad1)
- R30 pad 2: Net-(Q7-D) -> Net-(Q11-D)
- R32 pad 2: Net-(Q8-D) -> Net-(Q10-D)
- R36 pad 2: Net-(Q10-D) -> Net-(Q7-D)
- R38 pad 2: Net-(Q11-D) -> Net-(Q8-D)
- R41 pad 2: Net-(Q12-D) -> Net-(Q16-D)
- R43 pad 2: Net-(Q13-D) -> Net-(Q15-D)
- R47 pad 2: Net-(Q15-D) -> Net-(Q13-D)
- R49 pad 2: Net-(Q16-D) -> Net-(Q12-D)
- U12 pad 17: (no net) -> GND
- U2 pad 5: (no net) -> GND
- U3 pad 5: (no net) -> GND
- U4 pad 11: unconnected-(U4-THERM-Pad11) -> GND
- U5 pad 5: (no net) -> GND
- U6 pad 5: (no net) -> GND
- U7 pad 10: Net-(Q5-S) -> Net-(U7-SW2)
- U7 pad 21: Net-(Q3-S) -> Net-(U7-SW1)
- U7 pad 41: (no net) -> GND
- U8 pad 10: B_USB-C_BUCK_15V_SEL -> B_SUB-C_BUCK_P-GOOD
- U8 pad 11: B_USB-C_BUCK_12V_SEL -> B_USB-C_BUCK_EN
- U8 pad 13: B_USB-C_BUCK_9V_SEL -> F_USB-C_BUCK_EN
- U8 pad 14: B_USB-C_BUCK_5V_SEL -> F_USB-C_BUCK_5V_SEL
- U8 pad 15: F_USB-C_BUCK_EN -> F_USB-C_BUCK_9V_SEL
- U8 pad 16: B_USB-C_BUCK_EN -> F_USB-C_BUCK_12V_SEL
- U8 pad 17: F_SUB-C_BUCK_P-GOOD -> F_USB-C_BUCK_15V_SEL
- U8 pad 18: B_SUB-C_BUCK_P-GOOD -> F_USB-C_BUCK_20V_SEL
- U8 pad 20: CAN_SILENT -> ADC_ALERT
- U8 pad 4: F_USB-C_BUCK_20V_SEL -> B_USB-C_BUCK_5V_SEL
- U8 pad 5: F_USB-C_BUCK_15V_SEL -> B_USB-C_BUCK_9V_SEL
- U8 pad 6: F_USB-C_BUCK_12V_SEL -> B_USB-C_BUCK_12V_SEL
- U8 pad 7: F_USB-C_BUCK_9V_SEL -> B_USB-C_BUCK_15V_SEL
- U8 pad 8: F_USB-C_BUCK_5V_SEL -> B_USB-C_BUCK_20V_SEL
- U8 pad 9: B_USB-C_BUCK_20V_SEL -> F_SUB-C_BUCK_P-GOOD
- U9 pad 19: ADC_ALERT -> CAN_SILENT
Routing:
- net +5V: track 0.00 -> 128.7 mm, vias 0 -> 3
- net 21V_PGOOD: track 0.00 -> 74.3 mm, vias 0 -> 2
- net GND: track 15.6 -> 84.0 mm, vias 41 -> 96
- net F_USB-C_BUCK_OUT: track 0.00 -> 58.4 mm, vias 0 -> 5
- net B_USB-C_BUCK_OUT: track 0.00 -> 55.5 mm, vias 0 -> 3
- net +3V3: track 0.00 -> 52.3 mm, vias 0 -> 4
- net B_USB-C_CSN: track 0.00 -> 50.5 mm, vias 0 -> 13
- net ADC_ALERT: track 0.00 -> 45.8 mm, vias 0 -> 2
- net I2C_SDA: track 0.00 -> 43.5 mm, vias 0 -> 2
- net I2C_SCL: track 0.00 -> 42.3 mm, vias 0 -> 2
- net F_USB-C_CSN: track 0.00 -> 42.3 mm, vias 0 -> 2
- net 5V_CSN: track 0.00 -> 40.1 mm, vias 0 -> 4
- net B_SUB-C_BUCK_P-GOOD: track 0.00 -> 33.0 mm, vias 0 -> 3
- net F_SUB-C_BUCK_P-GOOD: track 0.00 -> 30.8 mm, vias 0 -> 3
- net F_USB-C_BUCK_20V_SEL: track 0.00 -> 28.2 mm
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- added copper zone on F.Cu, net +21V
- added copper zone on In2.Cu, net +21V
- added copper zone on F.Cu, net /5V USB-A AND MCU POWER/5V_SW
- added copper zone on F.Cu, net 5V_CSN
- added copper zone on F.Cu, net B_USB-C_BUCK_OUT
- added copper zone on F.Cu, net B_USB-C_CSN
- added copper zone on F.Cu, net F_USB-C_BUCK_OUT
- added copper zone on F.Cu, net F_USB-C_CSN
- added copper zone on F.Cu, net Net-(U7-SW1)
- added copper zone on F.Cu, net Net-(U7-SW2)

Commit message: working on routing still  finnished psu section
Parts:
- added JP19: ~, Jumper:SolderJumper-3_P1.3mm_Open_RoundedPad1.0x1.5mm_NumberLabels, B.Cu at (345.6, 113.1)
- JP3: moved to B.Cu
- moved J10 363.8 mm to (418.1, 71.7)
- moved U10 343.5 mm to (406.4, 79.7)
- moved C45 339.4 mm to (417.8, 84.2), turned to 180 degrees
- moved R57 336.0 mm to (417.8, 86.2), turned to 180 degrees
- moved R61 332.0 mm to (417.8, 80.1), turned to 180 degrees
- moved R60 331.7 mm to (417.8, 82.1), turned to 180 degrees
- moved R58 331.3 mm to (417.8, 88.2)
- moved C43 322.2 mm to (395.1, 73.2)
- moved C40 318.8 mm to (393.3, 97.8), turned to -90 degrees
- moved C42 317.2 mm to (391.7, 97.8), turned to -90 degrees
- moved C48 316.8 mm to (395.1, 90.1), turned to 180 degrees
- moved C47 316.7 mm to (395.1, 91.8), turned to 180 degrees
- moved R55 313.8 mm to (395.1, 75.0)
- moved R56 313.4 mm to (395.1, 82.2), turned to 180 degrees
- moved R54 313.2 mm to (395.1, 80.4)
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Connections:
- C24 pad 1: F_USB-C_BUCK_OUT -> B_USB-C_BUCK_OUT
- C38 pad 1: B_USB-C_BUCK_OUT -> F_USB-C_BUCK_OUT
- C46 pad 1: +5V -> Net-(JP19-C)
- L3 pad 1: F_USB-C_CSN -> B_USB-C_CSN
- L4 pad 2: B_USB-C_CSN -> F_USB-C_CSN
- Q10 pad 2: F_USB-C_BUCK_15V_SEL -> B_USB-C_BUCK_15V_SEL
- Q11 pad 2: F_USB-C_BUCK_20V_SEL -> B_USB-C_BUCK_20V_SEL
- Q12 pad 2: B_USB-C_BUCK_5V_SEL -> F_USB-C_BUCK_5V_SEL
- Q13 pad 2: B_USB-C_BUCK_9V_SEL -> F_USB-C_BUCK_9V_SEL
- Q14 pad 2: B_USB-C_BUCK_12V_SEL -> F_USB-C_BUCK_12V_SEL
- Q15 pad 2: B_USB-C_BUCK_15V_SEL -> F_USB-C_BUCK_15V_SEL
- Q16 pad 2: B_USB-C_BUCK_20V_SEL -> F_USB-C_BUCK_20V_SEL
- Q7 pad 2: F_USB-C_BUCK_9V_SEL -> B_USB-C_BUCK_9V_SEL
- Q8 pad 2: F_USB-C_BUCK_5V_SEL -> B_USB-C_BUCK_5V_SEL
- Q9 pad 2: F_USB-C_BUCK_12V_SEL -> B_USB-C_BUCK_12V_SEL
- R18 pad 1: F_USB-C_BUCK_OUT -> B_USB-C_BUCK_OUT
- R18 pad 2: F_USB-C_CSN -> B_USB-C_CSN
- R19 pad 2: F_SUB-C_BUCK_P-GOOD -> B_SUB-C_BUCK_P-GOOD
- R25 pad 1: B_SUB-C_BUCK_P-GOOD -> F_SUB-C_BUCK_P-GOOD
- R26 pad 1: B_USB-C_CSN -> F_USB-C_CSN
- R26 pad 2: B_USB-C_BUCK_OUT -> F_USB-C_BUCK_OUT
- R28 pad 1: F_USB-C_BUCK_OUT -> B_USB-C_BUCK_OUT
- R28 pad 2: F_USB-C_BUCK_FB -> B_USB-C_BUCK_FB
- R29 pad 1: F_USB-C_BUCK_FB -> B_USB-C_BUCK_FB
- R31 pad 1: F_USB-C_BUCK_FB -> B_USB-C_BUCK_FB
- R33 pad 1: F_USB-C_BUCK_FB -> B_USB-C_BUCK_FB
- R35 pad 1: F_USB-C_BUCK_FB -> B_USB-C_BUCK_FB
- R37 pad 1: F_USB-C_BUCK_FB -> B_USB-C_BUCK_FB
- R39 pad 1: B_USB-C_BUCK_OUT -> F_USB-C_BUCK_OUT
- R39 pad 2: B_USB-C_BUCK_FB -> F_USB-C_BUCK_FB
- R40 pad 1: B_USB-C_BUCK_FB -> F_USB-C_BUCK_FB
- R42 pad 1: B_USB-C_BUCK_FB -> F_USB-C_BUCK_FB
- R44 pad 1: B_USB-C_BUCK_FB -> F_USB-C_BUCK_FB
- R46 pad 1: B_USB-C_BUCK_FB -> F_USB-C_BUCK_FB
- R48 pad 1: B_USB-C_BUCK_FB -> F_USB-C_BUCK_FB
- R71 pad 1: F_USB-C_BUCK_OUT -> B_USB-C_BUCK_OUT
- R71 pad 2: F_USB-C_BUCK_OUT_ADC -> B_USB-C_BUCK_OUT_ADC
- R72 pad 1: F_USB-C_BUCK_OUT_ADC -> B_USB-C_BUCK_OUT_ADC
- R73 pad 1: F_USB-C_CSN -> B_USB-C_CSN
- R73 pad 2: F_USB-C_CSN_ADC -> B_USB-C_CSN_ADC
- R74 pad 1: F_USB-C_CSN_ADC -> B_USB-C_CSN_ADC
- R75 pad 1: B_USB-C_BUCK_OUT -> F_USB-C_BUCK_OUT
- R75 pad 2: B_USB-C_BUCK_OUT_ADC -> F_USB-C_BUCK_OUT_ADC
- R76 pad 1: B_USB-C_BUCK_OUT_ADC -> F_USB-C_BUCK_OUT_ADC
- R77 pad 1: B_USB-C_CSN -> F_USB-C_CSN
- R77 pad 2: B_USB-C_CSN_ADC -> F_USB-C_CSN_ADC
- R78 pad 1: B_USB-C_CSN_ADC -> F_USB-C_CSN_ADC
- U11 pad 3: +5V -> Net-(JP19-C)
- U12 pad 3: F_USB-C_BUCK_OUT_ADC -> B_USB-C_BUCK_OUT_ADC
- U12 pad 4: F_USB-C_CSN_ADC -> B_USB-C_CSN_ADC
- U12 pad 5: B_USB-C_BUCK_OUT_ADC -> F_USB-C_BUCK_OUT_ADC
- U12 pad 6: B_USB-C_CSN_ADC -> F_USB-C_CSN_ADC
- U7 pad 24: F_SUB-C_BUCK_P-GOOD -> B_SUB-C_BUCK_P-GOOD
- U7 pad 26: F_USB-C_BUCK_OUT -> B_USB-C_BUCK_OUT
- U7 pad 27: F_USB-C_CSN -> B_USB-C_CSN
- U7 pad 28: F_USB-C_BUCK_FB -> B_USB-C_BUCK_FB
- U7 pad 3: B_USB-C_BUCK_FB -> F_USB-C_BUCK_FB
- U7 pad 31: F_USB-C_BUCK_EN -> B_USB-C_BUCK_EN
- U7 pad 4: B_USB-C_CSN -> F_USB-C_CSN
- U7 pad 40: B_USB-C_BUCK_EN -> F_USB-C_BUCK_EN
- U7 pad 5: B_USB-C_BUCK_OUT -> F_USB-C_BUCK_OUT
- U7 pad 7: B_SUB-C_BUCK_P-GOOD -> F_SUB-C_BUCK_P-GOOD
- U8 pad 10: B_SUB-C_BUCK_P-GOOD -> F_SUB-C_BUCK_P-GOOD
- U8 pad 11: B_USB-C_BUCK_EN -> F_USB-C_BUCK_EN
- U8 pad 13: F_USB-C_BUCK_EN -> B_USB-C_BUCK_EN
- U8 pad 14: F_USB-C_BUCK_5V_SEL -> B_USB-C_BUCK_5V_SEL
- U8 pad 15: F_USB-C_BUCK_9V_SEL -> B_USB-C_BUCK_9V_SEL
- U8 pad 16: F_USB-C_BUCK_12V_SEL -> B_USB-C_BUCK_12V_SEL
- U8 pad 17: F_USB-C_BUCK_15V_SEL -> B_USB-C_BUCK_15V_SEL
- U8 pad 18: F_USB-C_BUCK_20V_SEL -> B_USB-C_BUCK_20V_SEL
- U8 pad 4: B_USB-C_BUCK_5V_SEL -> F_USB-C_BUCK_5V_SEL
- U8 pad 5: B_USB-C_BUCK_9V_SEL -> F_USB-C_BUCK_9V_SEL
- U8 pad 6: B_USB-C_BUCK_12V_SEL -> F_USB-C_BUCK_12V_SEL
- U8 pad 7: B_USB-C_BUCK_15V_SEL -> F_USB-C_BUCK_15V_SEL
- U8 pad 8: B_USB-C_BUCK_20V_SEL -> F_USB-C_BUCK_20V_SEL
- U8 pad 9: F_SUB-C_BUCK_P-GOOD -> B_SUB-C_BUCK_P-GOOD
- U9 pad 11: MODE_BTN -> unconnected-(U9-P0_7-Pad11)
- U9 pad 13: SRC_BTN -> unconnected-(U9-P1_0-Pad13)
- U9 pad 14: UNIT_BTN -> DFP_C_ATTACH_1
- U9 pad 15: DISP_IRQ -> HUB_VBUS_DET
- U9 pad 16: DFP_C_ATTACH_1 -> UFP_C_ATTACH_0
- U9 pad 17: HUB_VBUS_DET -> MODE_BTN
- U9 pad 18: UFP_C_ATTACH_0 -> SRC_BTN
- U9 pad 19: CAN_SILENT -> UNIT_BTN
- U9 pad 20: IOX1_INT -> DISP_IRQ
- U9 pad 4: IOX_0_P_0_0 -> IOX1_INT
- U9 pad 5: IOX_0_P_0_1 -> CAN_SILENT
- U9 pad 6: unconnected-(U9-P0_2-Pad6) -> IOX_0_P_0_1
- U9 pad 7: unconnected-(U9-P0_3-Pad7) -> IOX_0_P_0_0
Routing:
- net GND: track 84.0 -> 408.2 mm, vias 96 -> 167
- net +3V3: track 52.3 -> 207.6 mm, vias 4 -> 12
- net I2C_SDA: track 43.5 -> 181.7 mm, vias 2 -> 5
- net I2C_SCL: track 42.3 -> 177.4 mm, vias 2 -> 5
- net RST: track 0.00 -> 133.5 mm, vias 0 -> 4
- net IOX1_INT: track 1.64 -> 106.1 mm, vias 0 -> 4
- net CAR_12V_IN: track 37.7 -> 134.8 mm, vias 19 -> 20
- net CAN_RX: track 0.00 -> 91.9 mm, vias 0 -> 2
- net CAN_TX: track 0.00 -> 84.4 mm, vias 0 -> 2
- net IOX_0_P_0_0: track 0.00 -> 64.2 mm, vias 0 -> 1
- net CAN_SILENT: track 0.00 -> 56.8 mm
- net IOX_0_P_0_1: track 0.00 -> 55.9 mm, vias 0 -> 1
- net +5V: track 128.7 -> 163.5 mm, vias 3 -> 10
- net CAN_L: track 0.00 -> 22.7 mm
- net F_USB-C_BUCK_20V_SEL: track 28.2 -> 8.60 mm
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- added copper zone on F.Cu, net +5V
- added copper zone on In2.Cu, net +5V
- added copper zone on In2.Cu, net B_USB-C_BUCK_OUT
- added copper zone on In2.Cu, net F_USB-C_BUCK_OUT

Commit message: worked on usb port and display routing
Parts:
- added TP9: TestPoint, TestPoint:TestPoint_Pad_D1.5mm, F.Cu at (350.6, 62.0)
- D13, D14, D19, D20, D21, D22, D35, D8, JP10, JP11, JP12, JP14, JP15, JP16, JP17, JP9, TP4, TP5: moved to B.Cu
- moved D26 433.4 mm to (505.9, 112.0), turned to 180 degrees
- moved D27 429.9 mm to (505.9, 108.0), turned to 180 degrees
- moved D28 429.0 mm to (505.9, 104.0), turned to 180 degrees
- moved D29 428.2 mm to (505.9, 100.0), turned to 180 degrees
- moved D30 419.6 mm to (496.0, 112.0), turned to 180 degrees
- moved D31 416.1 mm to (496.0, 108.0), turned to 180 degrees
- moved D32 415.2 mm to (496.0, 104.0), turned to 180 degrees
- moved D33 414.4 mm to (496.0, 100.0), turned to 180 degrees
- moved D34 413.7 mm to (496.0, 96.0), turned to 180 degrees
- moved D25 408.5 mm to (482.8, 92.0), turned to 180 degrees
- moved C111 405.4 mm to (485.4, 98.4), turned to 180 degrees
- moved C110 402.7 mm to (482.1, 98.4)
- moved R100 398.1 mm to (478.8, 98.4)
- moved R99 395.3 mm to (475.6, 98.4), turned to 180 degrees
- moved D24 388.0 mm to (461.9, 92.0), turned to 180 degrees
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Connections:
- net Net-(J7-TX1+) renamed /BACK_UFP_USB_C_PORT/UFP_TXA_P
- net Net-(J7-TX1-) renamed /BACK_UFP_USB_C_PORT/UFP_TXA_N
- net Net-(J7-TX2+) renamed /BACK_UFP_USB_C_PORT/UFP_TXB_P
- net Net-(J7-TX2-) renamed /BACK_UFP_USB_C_PORT/UFP_TXB_N
- net Net-(J8-RX1+) renamed /FRONT_DFP_USB_C_PORT/DFP_RXB_P
- net Net-(J8-RX1-) renamed /FRONT_DFP_USB_C_PORT/DFP_RXB_N
- C103 pad 1: Net-(J8-TX2-) -> /FRONT_DFP_USB_C_PORT/DFP_RXA_N
- C103 pad 2: DFP_3_TXB_N -> DFP_3_RXA_N
- C104 pad 1: DFP_3_TXB_P -> DFP_3_RXA_P
- C104 pad 2: Net-(J8-TX2+) -> /FRONT_DFP_USB_C_PORT/DFP_RXA_P
- C82 pad 1: /USBA_PORTS/P4_RX_P -> /USBA_PORTS/P4_TX_P
- C82 pad 2: Net-(J4-STDA_SSRX+) -> /USBA_PORTS/P4_TXP_P
- C83 pad 1: Net-(J4-STDA_SSRX-) -> /USBA_PORTS/P4_TXP_N
- C83 pad 2: /USBA_PORTS/P4_RX_N -> /USBA_PORTS/P4_TX_N
- C84 pad 1: /USBA_PORTS/P2_RX_P -> /USBA_PORTS/P2_TX_P
- C84 pad 2: Net-(J3-STDA_SSRX+) -> /USBA_PORTS/P2_TXP_P
- C85 pad 1: Net-(J3-STDA_SSRX-) -> /USBA_PORTS/P2_TXP_N
- C85 pad 2: /USBA_PORTS/P2_RX_N -> /USBA_PORTS/P2_TX_N
- C86 pad 1: /USBA_PORTS/P5_RX_P -> /USBA_PORTS/P5_TX_P
- C86 pad 2: Net-(J6-STDA_SSRX+) -> /USBA_PORTS/P5_TXP_P
- C87 pad 1: Net-(J6-STDA_SSRX-) -> /USBA_PORTS/P5_TXP_N
- C87 pad 2: /USBA_PORTS/P5_RX_N -> /USBA_PORTS/P5_TX_N
- C88 pad 1: /USBA_PORTS/P3_RX_P -> /USBA_PORTS/P3_TX_P
- C88 pad 2: Net-(J5-STDA_SSRX+) -> /USBA_PORTS/P3_TXP_P
- C89 pad 1: Net-(J5-STDA_SSRX-) -> /USBA_PORTS/P3_TXP_N
- C89 pad 2: /USBA_PORTS/P3_RX_N -> /USBA_PORTS/P3_TX_N
- D13 pad 3: /USBA_PORTS/P5_2_N -> /USBA_PORTS/P5_RX_P
- D13 pad 4: /USBA_PORTS/P5_TX_P -> /USBA_PORTS/P5_RX_N
- D13 pad 5: /USBA_PORTS/P5_TX_N -> /USBA_PORTS/P5_TXP_P
- D13 pad 6: /USBA_PORTS/P5_RX_P -> /USBA_PORTS/P5_TXP_N
- D13 pad 7: /USBA_PORTS/P5_RX_N -> /USBA_PORTS/P5_2_N
- D14 pad 3: /USBA_PORTS/P3_2_N -> /USBA_PORTS/P3_RX_P
- D14 pad 4: /USBA_PORTS/P3_TX_P -> /USBA_PORTS/P3_RX_N
- D14 pad 5: /USBA_PORTS/P3_TX_N -> /USBA_PORTS/P3_TXP_P
- D14 pad 6: /USBA_PORTS/P3_RX_P -> /USBA_PORTS/P3_TXP_N
- D14 pad 7: /USBA_PORTS/P3_RX_N -> /USBA_PORTS/P3_2_N
- D19 pad 6: UFP_3_TXA_P -> UFP_3_TXA_N
- D19 pad 7: UFP_3_TXA_N -> UFP_3_TXA_P
- D21 pad 3: DFP_2_N -> DFP_3_RXB_P
- D21 pad 4: DFP_3_TXA_P -> DFP_3_RXB_N
- D21 pad 5: DFP_3_TXA_N -> DFP_3_TXB_N
- D21 pad 6: DFP_3_RXA_P -> DFP_3_TXB_P
- D21 pad 7: DFP_3_RXA_N -> DFP_2_N
- D22 pad 1: DFP_3_TXB_N -> DFP_CC2
- D22 pad 3: DFP_3_TXB_P -> DFP_3_RXA_P
- D22 pad 4: DFP_3_RXB_N -> DFP_3_RXA_N
- D22 pad 5: DFP_3_RXB_P -> DFP_3_TXA_N
- D22 pad 6: DFP_CC1 -> DFP_3_TXA_P
- D22 pad 7: DFP_CC2 -> DFP_CC1
- D35 pad 3: /USBA_PORTS/P4_2_N -> /USBA_PORTS/P4_RX_P
- D35 pad 4: /USBA_PORTS/P4_TX_P -> /USBA_PORTS/P4_RX_N
- D35 pad 5: /USBA_PORTS/P4_TX_N -> /USBA_PORTS/P4_TXP_P
- D35 pad 6: /USBA_PORTS/P4_RX_P -> /USBA_PORTS/P4_TXP_N
- D35 pad 7: /USBA_PORTS/P4_RX_N -> /USBA_PORTS/P4_2_N
- D8 pad 3: /USBA_PORTS/P2_2_N -> /USBA_PORTS/P2_RX_P
- D8 pad 4: /USBA_PORTS/P2_TX_P -> /USBA_PORTS/P2_RX_N
- D8 pad 5: /USBA_PORTS/P2_TX_N -> /USBA_PORTS/P2_TXP_P
- D8 pad 6: /USBA_PORTS/P2_RX_P -> /USBA_PORTS/P2_TXP_N
- D8 pad 7: /USBA_PORTS/P2_RX_N -> /USBA_PORTS/P2_2_N
- J3 pad 5: Net-(J3-STDA_SSRX-) -> /USBA_PORTS/P2_RX_N
- J3 pad 6: Net-(J3-STDA_SSRX+) -> /USBA_PORTS/P2_RX_P
- J3 pad 8: /USBA_PORTS/P2_TX_N -> /USBA_PORTS/P2_TXP_N
- J3 pad 9: /USBA_PORTS/P2_TX_P -> /USBA_PORTS/P2_TXP_P
- J4 pad 5: Net-(J4-STDA_SSRX-) -> /USBA_PORTS/P4_RX_N
- J4 pad 6: Net-(J4-STDA_SSRX+) -> /USBA_PORTS/P4_RX_P
- J4 pad 8: /USBA_PORTS/P4_TX_N -> /USBA_PORTS/P4_TXP_N
- J4 pad 9: /USBA_PORTS/P4_TX_P -> /USBA_PORTS/P4_TXP_P
- J5 pad 5: Net-(J5-STDA_SSRX-) -> /USBA_PORTS/P3_RX_N
- J5 pad 6: Net-(J5-STDA_SSRX+) -> /USBA_PORTS/P3_RX_P
- J5 pad 8: /USBA_PORTS/P3_TX_N -> /USBA_PORTS/P3_TXP_N
- J5 pad 9: /USBA_PORTS/P3_TX_P -> /USBA_PORTS/P3_TXP_P
- J6 pad 5: Net-(J6-STDA_SSRX-) -> /USBA_PORTS/P5_RX_N
- J6 pad 6: Net-(J6-STDA_SSRX+) -> /USBA_PORTS/P5_RX_P
- J6 pad 8: /USBA_PORTS/P5_TX_N -> /USBA_PORTS/P5_TXP_N
- J6 pad 9: /USBA_PORTS/P5_TX_P -> /USBA_PORTS/P5_TXP_P
- J8 pad A10: DFP_3_RXA_N -> /FRONT_DFP_USB_C_PORT/DFP_RXA_N
- J8 pad A11: DFP_3_RXA_P -> /FRONT_DFP_USB_C_PORT/DFP_RXA_P
- J8 pad B2: Net-(J8-TX2+) -> DFP_3_TXB_P
- J8 pad B3: Net-(J8-TX2-) -> DFP_3_TXB_N
- JP11 pad 1: +3V3 -> +5V
- JP11 pad 3: +5V -> +3V3
- JP16 pad 1: +3V3 -> +5V
- JP16 pad 3: +5V -> +3V3
- Q18 pad 2: Net-(Q18-G) -> UFP_VBUS
- Q18 pad 3: Net-(Q18-S) -> Net-(Q18-G)
- Q18 pad 4: (no net) -> Net-(Q18-S-Pad4)
- Q18 pad 5: (no net) -> UFP_VBUS
- Q18 pad 6: (no net) -> UFP_VBUS
- Q18 pad 7: (no net) -> UFP_VBUS
- Q18 pad 8: (no net) -> Net-(Q18-S-Pad4)
- Q19 pad 2: Net-(Q19-G) -> UFP_VBUS
- Q19 pad 3: Net-(Q19-S) -> Net-(Q19-G)
- Q19 pad 4: (no net) -> Net-(Q19-S-Pad4)
- Q19 pad 5: (no net) -> UFP_VBUS
- Q19 pad 6: (no net) -> UFP_VBUS
- Q19 pad 7: (no net) -> UFP_VBUS
- Q19 pad 8: (no net) -> Net-(Q19-S-Pad4)
- Q20 pad 2: Net-(Q18-G) -> Net-(JP13-C)
- Q20 pad 3: Net-(Q18-S) -> Net-(Q19-G)
- Q20 pad 4: (no net) -> Net-(Q19-S-Pad4)
- Q20 pad 5: (no net) -> Net-(JP13-C)
- Q20 pad 6: (no net) -> Net-(JP13-C)
- Q20 pad 7: (no net) -> Net-(JP13-C)
- Q20 pad 8: (no net) -> Net-(Q19-S-Pad4)
- Q21 pad 2: Net-(Q19-G) -> B_USB-C_BUCK_OUT
- Q21 pad 3: Net-(Q19-S) -> Net-(Q18-G)
- Q21 pad 4: (no net) -> Net-(Q18-S-Pad4)
- Q21 pad 5: (no net) -> B_USB-C_BUCK_OUT
- Q21 pad 6: (no net) -> B_USB-C_BUCK_OUT
- Q21 pad 7: (no net) -> B_USB-C_BUCK_OUT
- Q21 pad 8: (no net) -> Net-(Q18-S-Pad4)
- Q22 pad 2: Net-(Q22-G) -> DFP_VBUS
- Q22 pad 3: Net-(Q22-S) -> Net-(Q22-G)
- Q22 pad 4: (no net) -> Net-(Q22-S-Pad4)
- Q22 pad 5: (no net) -> DFP_VBUS
- Q22 pad 6: (no net) -> DFP_VBUS
- Q22 pad 7: (no net) -> DFP_VBUS
- Q22 pad 8: (no net) -> Net-(Q22-S-Pad4)
- Q23 pad 2: Net-(Q23-G) -> DFP_VBUS
- Q23 pad 3: Net-(Q23-S) -> Net-(Q23-G)
- Q23 pad 4: (no net) -> Net-(Q23-S-Pad4)
- Q23 pad 5: (no net) -> DFP_VBUS
- Q23 pad 6: (no net) -> DFP_VBUS
- Q23 pad 7: (no net) -> DFP_VBUS
- Q23 pad 8: (no net) -> Net-(Q23-S-Pad4)
- Q24 pad 2: Net-(Q22-G) -> Net-(JP18-C)
- Q24 pad 3: Net-(Q22-S) -> Net-(Q22-G)
- Q24 pad 4: (no net) -> Net-(Q22-S-Pad4)
- Q24 pad 5: (no net) -> Net-(JP18-C)
- Q24 pad 6: (no net) -> Net-(JP18-C)
- Q24 pad 7: (no net) -> Net-(JP18-C)
- Q24 pad 8: (no net) -> Net-(Q22-S-Pad4)
- Q25 pad 2: Net-(Q23-G) -> F_USB-C_BUCK_OUT
- Q25 pad 3: Net-(Q23-S) -> Net-(Q23-G)
- Q25 pad 4: (no net) -> Net-(Q23-S-Pad4)
- Q25 pad 5: (no net) -> F_USB-C_BUCK_OUT
- Q25 pad 6: (no net) -> F_USB-C_BUCK_OUT
- Q25 pad 7: (no net) -> F_USB-C_BUCK_OUT
- Q25 pad 8: (no net) -> Net-(Q23-S-Pad4)
- R90 pad 2: Net-(Q18-G) -> Net-(Q19-G)
- R91 pad 2: Net-(Q19-G) -> Net-(Q18-G)
- R92 pad 1: Net-(Q18-S) -> Net-(Q19-S-Pad4)
- R92 pad 2: Net-(Q18-G) -> Net-(Q19-G)
- R93 pad 1: Net-(Q19-S) -> Net-(Q18-S-Pad4)
- R93 pad 2: Net-(Q19-G) -> Net-(Q18-G)
- R97 pad 1: Net-(Q22-S) -> Net-(Q22-S-Pad4)
- R98 pad 1: Net-(Q23-S) -> Net-(Q23-S-Pad4)
- U13 pad 70: unconnected-(U13E-PRT_CTL1/GPIO17-Pad70) -> Net-(U13E-PRT_CTL1/GPIO17)
- U13 pad 73: (no net) -> DFP_C_ATTACH_1
- U13 pad 76: DFP_C_ATTACH_1 -> UFP_C_ATTACH_0
- U15 pad 16: (no net) -> unconnected-(U15-SPI_MISO-Pad16)
- U15 pad 21: (no net) -> GND
- U15 pad 6: unconnected-(U15-DBGACC_FOUND-Pad6) -> UFP_DBGACC
- U15 pad 7: (no net) -> unconnected-(U15-SPI_CS-Pad7)
- U16 pad 1: Net-(JP17-B) -> Net-(JP17-A)
- U16 pad 16: (no net) -> unconnected-(U16-SPI_MISO-Pad16)
- U16 pad 20: Net-(JP17-A) -> Net-(JP17-B)
- U16 pad 21: (no net) -> GND
- U16 pad 6: unconnected-(U16-DBGACC_FOUND-Pad6) -> DFP_DBGACC
- U16 pad 7: (no net) -> unconnected-(U16-SPI_CS-Pad7)
- U9 pad 10: unconnected-(U9-P0_6-Pad10) -> HUB_VBUS_DET
- U9 pad 11: unconnected-(U9-P0_7-Pad11) -> UFP_C_ATTACH_0
- U9 pad 14: DFP_C_ATTACH_1 -> unconnected-(U9-P1_1-Pad14)
- U9 pad 15: HUB_VBUS_DET -> DFP_DBGACC
- U9 pad 16: UFP_C_ATTACH_0 -> UFP_DBGACC
- U9 pad 17: MODE_BTN -> DISP_IRQ
- U9 pad 18: SRC_BTN -> MODE_BTN
- U9 pad 20: DISP_IRQ -> SRC_BTN
- U9 pad 9: unconnected-(U9-P0_5-Pad9) -> DFP_C_ATTACH_1
Routing:
- net +3V3: track 207.6 -> 496.6 mm, vias 12 -> 25
- net GND: track 408.2 -> 612.7 mm, vias 167 -> 209
- net DISP_IRQ: track 0.00 -> 191.4 mm, vias 0 -> 3
- net I2C_SDA: track 181.7 -> 341.8 mm, vias 5 -> 10
- net I2C_SCL: track 177.4 -> 322.6 mm, vias 5 -> 10
- net DFP_DBGACC: track 0.00 -> 123.7 mm, vias 0 -> 2
- net MODE_BTN: track 0.00 -> 122.9 mm
- net UNIT_BTN: track 0.00 -> 110.4 mm
- net SRC_BTN: track 0.00 -> 98.0 mm
- net DISP_SEG_D: track 0.00 -> 94.4 mm
- net DISP_DIG_7: track 0.00 -> 93.5 mm, vias 0 -> 2
- net DISP_SEG_A: track 0.00 -> 75.2 mm, vias 0 -> 2
- net DISP_SEG_E: track 0.00 -> 69.7 mm
- net +5V: track 163.5 -> 231.0 mm, vias 10 -> 14
- net DFP_2_P: track 0.00 -> 56.2 mm, vias 0 -> 4
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- added copper zone on F.Cu, net DFP_VBUS
- added copper zone on In2.Cu, net DFP_VBUS
- added copper zone on F.Cu, net Net-(JP13-C)
- added copper zone on F.Cu, net Net-(JP18-C)
- added copper zone on F.Cu, net Net-(Q18-S-Pad4)
- added copper zone on F.Cu, net Net-(Q19-S-Pad4)
- added copper zone on F.Cu, net Net-(Q22-S-Pad4)
- added copper zone on F.Cu, net Net-(Q23-S-Pad4)
- added copper zone on F.Cu, net UFP_VBUS
- added copper zone on In2.Cu, net UFP_VBUS
Other:
- board outline added: 175 x 139 mm
- board text added: "100W"
- board text added: "10W"
- board text added: "20W"
- board text added: "40W"
- board text added: "65W"
- board text added: "AMPS"
- board text added: "BACK C"
- board text added: "FRONT C"
- board text added: "SYSTEM"
- board text added: "USB A"
- board text added: "VOLTS"
- board text added: "WATTS"

Commit message: working in final routing
Parts:
- C53, C54, C55, C56, C59, C60, C61, C62, C63, C64, C65, C66, C67, C68, C69, C70, C71, C72, C73, C74, C75, C76, C77, C78, JP4, JP5, JP6, JP7, JP8, TP1, TP3, TP9: moved to B.Cu
- moved Q15 345.0 mm to (157.4, 124.0)
- moved R48 345.0 mm to (166.4, 114.2)
- moved C1 345.0 mm to (129.6, 77.2)
- moved C10 345.0 mm to (114.7, 75.2)
- moved C101 345.0 mm to (81.1, 159.5)
- moved C104 345.0 mm to (95.0, 159.5)
- moved C105 345.0 mm to (88.6, 132.9)
- moved C106 345.0 mm to (87.0, 132.9)
- moved C108 345.0 mm to (91.8, 132.9)
- moved C109 345.0 mm to (87.1, 143.2)
- moved C11 345.0 mm to (114.7, 73.6)
- moved C110 345.0 mm to (140.6, 147.8)
- moved C112 345.0 mm to (118.6, 33.7)
- moved C113 345.0 mm to (114.7, 71.9)
- moved C19 345.0 mm to (114.0, 81.2)
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Connections:
- J3 pad S: (no net) -> GNDS
- U13 pad 101: (no net) -> GND
- U13 pad 28: /USBA_PORTS/P2_2_P -> /USBA_PORTS/P5_2_P
- U13 pad 29: /USBA_PORTS/P2_2_N -> /USBA_PORTS/P5_2_N
- U13 pad 30: /USBA_PORTS/P2_TX_P -> /USBA_PORTS/P5_TX_P
- U13 pad 31: /USBA_PORTS/P2_TX_N -> /USBA_PORTS/P5_TX_N
- U13 pad 33: /USBA_PORTS/P2_RX_P -> /USBA_PORTS/P5_RX_P
- U13 pad 34: /USBA_PORTS/P2_RX_N -> /USBA_PORTS/P5_RX_N
- U13 pad 35: /USBA_PORTS/P3_2_P -> /USBA_PORTS/P2_2_P
- U13 pad 36: /USBA_PORTS/P3_2_N -> /USBA_PORTS/P2_2_N
- U13 pad 37: /USBA_PORTS/P3_TX_P -> /USBA_PORTS/P2_TX_P
- U13 pad 38: /USBA_PORTS/P3_TX_N -> /USBA_PORTS/P2_TX_N
- U13 pad 40: /USBA_PORTS/P3_RX_P -> /USBA_PORTS/P2_RX_P
- U13 pad 41: /USBA_PORTS/P3_RX_N -> /USBA_PORTS/P2_RX_N
- U13 pad 43: /USBA_PORTS/P4_2_P -> /USBA_PORTS/P3_2_P
- U13 pad 44: /USBA_PORTS/P4_2_N -> /USBA_PORTS/P3_2_N
- U13 pad 45: /USBA_PORTS/P4_TX_P -> /USBA_PORTS/P3_TX_P
- U13 pad 46: /USBA_PORTS/P4_TX_N -> /USBA_PORTS/P3_TX_N
- U13 pad 48: /USBA_PORTS/P4_RX_P -> /USBA_PORTS/P3_RX_P
- U13 pad 49: /USBA_PORTS/P4_RX_N -> /USBA_PORTS/P3_RX_N
- U13 pad 51: Net-(D16-A) -> Net-(D10-A)
- U13 pad 52: Net-(D10-A) -> Net-(D15-A)
- U13 pad 57: Net-(D15-A) -> Net-(D9-A)
- U13 pad 58: Net-(D9-A) -> Net-(D16-A)
- U13 pad 74: (no net) -> I2C_SDA
- U13 pad 8: unconnected-(U13E-USB3DN_TXDP1A-Pad8) -> DFP_3_TXA_P
- U13 pad 86: /USBA_PORTS/P5_2_P -> /USBA_PORTS/P4_2_P
- U13 pad 87: /USBA_PORTS/P5_2_N -> /USBA_PORTS/P4_2_N
- U13 pad 88: /USBA_PORTS/P5_TX_P -> /USBA_PORTS/P4_TX_P
- U13 pad 89: /USBA_PORTS/P5_TX_N -> /USBA_PORTS/P4_TX_N
- U13 pad 9: unconnected-(U13E-USB3DN_TXDM1A-Pad9) -> DFP_3_TXA_N
- U13 pad 91: /USBA_PORTS/P5_RX_P -> /USBA_PORTS/P4_RX_P
- U13 pad 92: /USBA_PORTS/P5_RX_N -> /USBA_PORTS/P4_RX_N
Routing:
- net +5V: track 231.0 -> 392.5 mm, vias 14 -> 19
- net DFP_3_RXA_N: track 33.1 -> 149.4 mm, vias 1 -> 4
- net DFP_2_P: track 56.2 -> 164.8 mm, vias 4 -> 6
- net DFP_2_N: track 54.2 -> 162.6 mm, vias 4 -> 6
- net DFP_3_TXA_P: track 39.3 -> 145.5 mm, vias 1 -> 3
- net DFP_3_TXA_N: track 38.5 -> 144.7 mm, vias 1 -> 3
- net Net-(D15-A): track 0.00 -> 104.0 mm, vias 0 -> 2
- net DFP_3_RXA_P: track 33.1 -> 136.1 mm, vias 1 -> 4
- net Net-(D9-A): track 0.00 -> 100.0 mm, vias 0 -> 2
- net HUB_VBUS_DET: track 0.00 -> 99.7 mm, vias 0 -> 2
- net DFP_3_TXB_P: track 31.7 -> 127.6 mm, vias 1 -> 3
- net DFP_3_TXB_N: track 31.2 -> 127.1 mm, vias 1 -> 3
- net DFP_3_RXB_P: track 20.5 -> 113.0 mm, vias 1 -> 4
- net DFP_3_RXB_N: track 20.4 -> 112.9 mm, vias 1 -> 4
- net /USBA_PORTS/P2_2_P: track 4.32 -> 86.3 mm, vias 0 -> 2
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- added copper zone on In2.Cu, net +1V2
- added copper zone on In2.Cu, net +3V3
Other:
- board size 175 x 139 mm -> 150.1 x 139 mm

Commit message: finaliseing pcb layout will come back later for a fresh look
Parts:
- moved R104 5.10 mm to (122.8, 33.3), turned to 90 degrees
- moved C112 2.62 mm to (121.2, 33.3), turned to 90 degrees
Connections:
- J4 pad S: (no net) -> GNDS
- J5 pad S: (no net) -> GNDS
- J6 pad S: (no net) -> GNDS
Routing:
- net GNDS: track 0.00 -> 410.6 mm, vias 0 -> 1
- net F_USB-C_BUCK_FB: track 9.10 -> 23.8 mm
- net GND: track 692.5 -> 701.6 mm, vias 219 -> 233
- net +21V: track 42.6 -> 51.1 mm, vias 26 -> 27
- added copper zone on B.Cu, net /12-21V INPUT BOOST CONVERTER/SW
- added copper zone on In1.Cu, net GND
