File: hardware/usbc-car-module.kicad_pcb (KiCad board)
At the start: 4 copper layers, 150.1 x 139 mm, 350 parts, among them J10 PROG_PORT, J3 0483930003, J4 0483930003, J5 0483930003, J6 0483930003, J7 USB4200-03-A (VIRT FLAG MOUNT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, J8 USB4200-03-A (VIRT FLAG MOUNT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, J9 684M7W2103L461, Q1 NMOS, Q10 NMOS, Q11 NMOS, Q12 NMOS, Q13 NMOS, Q14 NMOS, Q15 NMOS, Q16 NMOS, Q17 BC847BS-7-F, Q18 PMOS, Q19 PMOS, Q2 NMOS, Q20 PMOS, Q21 PMOS, Q22 PMOS, Q23 PMOS, Q24 PMOS, Q25 PMOS, Q26 NMOS, Q27 AON7421, Q3 PMPB11EN,115, Q4 PMPB11EN,115, Q5 PMPB11EN,115, Q6 PMPB11EN,115, Q7 NMOS, Q8 NMOS, Q9 NMOS, SW1 SW_Push, SW2 SW_Push, SW3 SW_Push, U1 LM51231-Q1, U10 ESP-12F, U11 MCP2558FD-xMF, U14 CP2102N-QFN20, U17 AS1115-BSST, U18 LTC-5723HR, U19 NCP177BMX330TCG, U2 NCP177BMX330TCG, U3 NCP177BMX330TCG, U4 LMR14050-Q1, U5 NCP177AMX120TCG, U6 NCP177AMX120TCG, U8 PI4IOE5V6416LEX, U9 PI4IOE5V6416LEX, Y1 25MHz

Commit message: messing arround with pcb to finalise
Parts:
- added REF**: OSHW-Logo2_7.3x6mm_SilkScreen, Symbol:OSHW-Logo2_7.3x6mm_SilkScreen, F.Cu at (33.0, 38.0)
- added TP10: TestPoint, TestPoint:TestPoint_Pad_D1.5mm, F.Cu at (113.5, 102.0)
- added TP11: TestPoint, TestPoint:TestPoint_Pad_D1.5mm, F.Cu at (113.5, 113.0)
- added TP12: TestPoint, TestPoint:TestPoint_Pad_D1.5mm, F.Cu at (112.5, 86.5)
- added TP13: TestPoint, TestPoint:TestPoint_Pad_D1.5mm, F.Cu at (138.5, 100.0)
- moved R28 2.55 mm to (119.5, 113.7)
- moved R29 2.55 mm to (121.2, 113.7)
- moved R31 2.55 mm to (122.9, 113.7)
- moved R33 2.55 mm to (124.5, 113.7)
- moved R35 2.55 mm to (126.2, 113.7)
- moved R37 2.55 mm to (127.8, 113.7)
- moved TP1 0.51 mm to (50.0, 85.6)
Routing:
- net +3V3: track 563.9 -> 462.4 mm
- net +1V2: track 120.5 -> 47.1 mm
- net +5V: track 392.5 -> 399.2 mm
- net +21V: track 51.1 -> 54.9 mm
- net Net-(R29-Pad2): track 5.25 -> 8.26 mm
- net B_USB-C_BUCK_FB: track 22.0 -> 19.5 mm
- net Net-(R37-Pad2): track 6.95 -> 4.74 mm
- net F_USB-C_BUCK_OUT: track 55.5 -> 57.0 mm, vias 16 -> 17
- net Net-(R31-Pad2): track 4.00 -> 5.44 mm
- net Net-(R35-Pad2): track 4.70 -> 3.62 mm
- net B_USB-C_BUCK_OUT: track 58.1 -> 57.0 mm, vias 19 -> 20
- net Net-(JP16-C): track 26.1 -> 27.1 mm
- net GND: vias 233 -> 234
Other:
- board text added: "+1.2V"
- board text added: "+21V"
- board text added: "+3.3V"
- board text added: "+5V"
- board text added: "12V"
- board text added: "15V"
- board text added: "20V"
- board text added: "5V"
- board text added: "9V"
- board text added: "ALT_MUX_EN/GPIO_70"
- board text added: "BACK"
- board text added: "CAN TERM RES"
- board text added: "CAN VDD"
- board text added: "CC_POL/GPIO_71"
- board text added: "DFP EN_USBFETx"
- board text added: "DFP VCONN_IN VOLTAGE SEL"
- board text added: "DFP_CC_CRTL"
- board text added: "FRONT"
- board text added: "GND"
- board text added: "GPIO"
- board text added: "HT_0/GPIO_23"
- board text added: "HT_1/GPIO_67"
- board text added: "HUB RST"
- board text added: "HUB RST LINE"
- board text added: "I2C"
- board text added: "IO0"
- board text added: "MODE"
- board text added: "PRT_CTL_1/GPIO_17"
- board text added: "PRT_CTL_6/GPIO_18"
- board text added: "REV A"
- board text added: "RST"
- board text added: "RX"
- board text added: "SOURCE"
- board text added: "SYNC OUT"
- board text added: "TX"
- board text added: "UART RST"
- board text added: "UFP EN_USBFETx"
- board text added: "UFP VCONN_IN VOLTAGE SEL"
- board text added: "UFP_CC_CRTL"
- board text added: "UNITS"
- board text added: "V_BACK"
- board text added: "V_FRONT"
