File: hardware/USB_UART.kicad_sch (KiCad schematic)
At the start: 14 parts, among them Q17 BC847BS-7-F, U14 CP2102N-QFN20

Commit message: working in final routing
Changed lines of the file:
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@@
   (symbol (lib_id "CARTHING:USB5916C") (at 71.12 87.63 0) (unit 10)
     (in_bom yes) (on_board yes) (dnp no) (fields_autoplaced)
-    (property "Reference" "U13" (at 71.755 75.2381 0)
+    (property "Reference" "U13" (at 69.85 75.2381 0)
       (effects (font (size 1.27 1.27)))
     )
@@
     )
     (pin "10")
+    (pin "101")
     (pin "17")
     (pin "2")
@@
     (pin "93")
     (pin "98")
-    (pin "EP")
     (pin "1")
     (pin "20")
@@
     (pin "7")
     (pin "70")
-    (pin "76")
+    (pin "73")
     (pin "8")
     (pin "9")
@@
           (reference "U13") (unit 10)
         )
+        (path "/fae025e9-99c5-40c1-af6f-99dc1edbfa43/7a7a6512-c96f-448a-bb8d-4d6e185adf7f"
+          (reference "U13") (unit 10)
+        )

Commit message: finaliseing pcb layout will come back later for a fresh look
Other:
- company: (none) -> MICK MAKE
- title: (none) -> 200W USB PD 3.1 HUB
Changed lines of the file:
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@@
 (kicad_sch (version 20230121) (generator eeschema)
   (paper "A4")
+  (title_block
+    (title "200W USB PD 3.1 HUB")
+    (date "2023-10-03")
+    (rev "A")
+    (company "MICK MAKE")
+    (comment 1 "THIS IS A 2X 100W USB PD SOURCE ")
+    (comment 2 "HUB USB SPEC 3.1")
+    (comment 3 "TOTAL SYSTEM POWER IS ~275w")
+  )
   (junction (at 110.49 44.45) (diameter 0) (color 0 0 0 0)
   )

Commit message: ned to fix port swap before  prod
Parts:
- added SW1: SW_SPDT, CARTHING:A107673, symbol Switch:SW_SPDT
Connections:
- net GND: now also SW1.3 (C)
- net UART_RST: now also SW1.2 (B)
Changed lines of the file:
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@@
   (junction (at 130.81 57.15) (diameter 0) (color 0 0 0 0)
+  )
+  (junction (at 74.93 63.5) (diameter 0) (color 0 0 0 0)
   )
   (junction (at 69.85 63.5) (diameter 0) (color 0 0 0 0)
@@
     (stroke (width 0) (type default))
   )
+  (wire (pts (xy 74.93 63.5) (xy 80.01 63.5))
+    (stroke (width 0) (type default))
+  )
   (wire (pts (xy 119.38 78.74) (xy 95.25 78.74))
     (stroke (width 0) (type default))
@@
     (stroke (width 0) (type default))
   )
+  (wire (pts (xy 74.93 53.34) (xy 74.93 63.5))
+    (stroke (width 0) (type default))
+  )
   (wire (pts (xy 110.49 55.88) (xy 121.92 55.88))
     (stroke (width 0) (type default))
@@
     (stroke (width 0) (type default))
   )
-  (wire (pts (xy 69.85 63.5) (xy 80.01 63.5))
+  (wire (pts (xy 69.85 63.5) (xy 74.93 63.5))
     (stroke (width 0) (type default))
   )
@@
   )
   (wire (pts (xy 104.14 55.88) (xy 110.49 55.88))
+    (stroke (width 0) (type default))
+  )
+  (wire (pts (xy 72.39 40.64) (xy 72.39 43.18))
     (stroke (width 0) (type default))
   )
@@
     )
   )
+  (symbol (lib_id "Switch:SW_SPDT") (at 74.93 48.26 270) (mirror x) (unit 1)
+    (in_bom yes) (on_board yes) (dnp no)
+    (property "Reference" "SW1" (at 71.12 48.26 90)
+      (effects (font (size 1.27 1.27)))
+    )
+    (property "Value" "SW_SPDT" (at 78.74 48.26 0)
+      (effects (font (size 1.27 1.27)) hide)
+    )
+    (property "Footprint" "CARTHING:A107673" (at 74.93 48.26 0)
+      (effects (font (size 1.27 1.27)) hide)
+    )
+    (property "Datasheet" "~" (at 74.93 48.26 0)
+      (effects (font (size 1.27 1.27)) hide)
+    )
+    (pin "1")
+    (pin "2")
+    (pin "3")
+    (instances
+      (project "bno085"
+        (path "/4a81f164-327a-47fd-b6e9-9a19456d34d9"
+          (reference "SW1") (unit 1)
+        )
+      )
+      (project "usbc-car-module"
+        (path "/fae025e9-99c5-40c1-af6f-99dc1edbfa43/115036d9-3633-4f5d-a259-54a6f0cf58ce"
+          (reference "SW4") (unit 1)
+        )
+      )
+    )
+  )
   (symbol (lib_id "power:GND") (at 104.14 57.15 0) (unit 1)
     (in_bom yes) (on_board yes) (dnp no) (fields_autoplaced)
@@
         )
       )
+    )
+  )
+  (symbol (lib_id "power:GND") (at 72.39 40.64 180) (unit 1)
+    (in_bom yes) (on_board yes) (dnp no) (fields_autoplaced)
+    (property "Reference" "#PWR0152" (at 72.39 34.29 0)
+      (effects (font (size 1.27 1.27)) hide)
+    )
+    (property "Value" "GND" (at 72.39 37.1381 0)
+      (effects (font (size 1.27 1.27)))
+    )
+    (property "Footprint" "" (at 72.39 40.64 0)
+      (effects (font (size 1.27 1.27)) hide)
+    )
+    (property "Datasheet" "" (at 72.39 40.64 0)
+      (effects (font (size 1.27 1.27)) hide)
+    )
+    (pin "1")
+    (instances
+      (project "usbc-car-module"
+        (path "/fae025e9-99c5-40c1-af6f-99dc1edbfa43/115036d9-3633-4f5d-a259-54a6f0cf58ce"
+          (reference "#PWR0152") (unit 1)
+        )
+      )
