File: hardware/F_AND_B_VOUT_FEEDBACK_NETWORKS.kicad_sch (KiCad schematic)
At the start: 32 parts, among them Q10 NMOS, Q11 NMOS, Q7 NMOS, Q8 NMOS, Q9 NMOS

Commit message: finnished rudimentry schimatics still needs alot of work
Connections:
- net B_USB-C_BUCK_12V_SEL: now also Q9.2 (G)
- net B_USB-C_BUCK_15V_SEL: now also Q8.2 (G)
- net B_USB-C_BUCK_20V_SEL: now also Q7.2 (G)
- net B_USB-C_BUCK_5V_SEL: now also Q11.2 (G)
- net B_USB-C_BUCK_9V_SEL: now also Q10.2 (G)
- net F_USB-C_BUCK_12V_SEL: now also Q9.2 (G)
- net F_USB-C_BUCK_15V_SEL: now also Q8.2 (G)
- net F_USB-C_BUCK_20V_SEL: now also Q7.2 (G)
- net F_USB-C_BUCK_5V_SEL: now also Q11.2 (G)
- net F_USB-C_BUCK_9V_SEL: now also Q10.2 (G)
Changed lines of the file:
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@@
+    (stroke (width 0) (type default))
+  )
+  (wire (pts (xy 182.88 110.49) (xy 182.88 111.76))
     (stroke (width 0) (type default))
   )
   (wire (pts (xy 36.83 80.01) (xy 36.83 82.55))
+    (stroke (width 0) (type default))
+  )
+  (wire (pts (xy 44.45 118.11) (xy 44.45 119.38))
     (stroke (width 0) (type default))
   )
@@
     (stroke (width 0) (type default))
   )
+  (wire (pts (xy 213.36 110.49) (xy 213.36 111.76))
+    (stroke (width 0) (type default))
+  )
   (wire (pts (xy 205.74 91.44) (xy 205.74 93.98))
     (stroke (width 0) (type default))
   )
   (wire (pts (xy 78.74 82.55) (xy 97.79 82.55))
+    (stroke (width 0) (type default))
+  )
+  (wire (pts (xy 201.93 116.84) (xy 201.93 118.11))
     (stroke (width 0) (type default))
   )
@@
     (stroke (width 0) (type default))
   )
+  (wire (pts (xy 55.88 111.76) (xy 55.88 113.03))
+    (stroke (width 0) (type default))
+  )
   (wire (pts (xy 194.31 101.6) (xy 194.31 111.76))
     (stroke (width 0) (type default))
@@
     (stroke (width 0) (type default))
   )
+  (wire (pts (xy 86.36 111.76) (xy 86.36 113.03))
+    (stroke (width 0) (type default))
+  )
+  (wire (pts (xy 171.45 116.84) (xy 171.45 118.11))
+    (stroke (width 0) (type default))
+  )
   (wire (pts (xy 48.26 149.86) (xy 36.83 149.86))
+    (stroke (width 0) (type default))
+  )
+  (wire (pts (xy 105.41 118.11) (xy 105.41 119.38))
     (stroke (width 0) (type default))
   )
@@
   )
   (wire (pts (xy 194.31 81.28) (xy 205.74 81.28))
+    (stroke (width 0) (type default))
+  )
+  (wire (pts (xy 74.93 118.11) (xy 74.93 119.38))
     (stroke (width 0) (type default))
   )
@@
     (stroke (width 0) (type default))
   )
+  (wire (pts (xy 232.41 116.84) (xy 232.41 118.11))
+    (stroke (width 0) (type default))
+  )

Commit message: working on hardware
Parts:
- Q10, Q11, Q7, Q8, Q9: footprint (none) -> Package_TO_SOT_SMD:SOT-416

Commit message: working assighning footprints still
Parts:
- R24, R25, R26, R27, R28, R29, R33: footprint (none) -> Resistor_SMD:R_0603_1608Metric
- R29, R30, R31, R32, R34: footprint (none) -> Potentiometer_SMD:Potentiometer_Bourns_TC33X_Vertical
Changed lines of the file:
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@@
       (effects (font (size 1.27 1.27)) (justify left))
     )
-    (property "Footprint" "" (at 35.052 88.9 90)
+    (property "Footprint" "Resistor_SMD:R_0603_1608Metric" (at 35.052 88.9 90)
       (effects (font (size 1.27 1.27)) hide)
     )
@@
       (effects (font (size 1.27 1.27)) (justify left))
     )
-    (property "Footprint" "" (at 46.482 88.9 90)
+    (property "Footprint" "Resistor_SMD:R_0603_1608Metric" (at 46.482 88.9 90)
       (effects (font (size 1.27 1.27)) hide)
     )
@@
       (effects (font (size 1.27 1.27)) (justify left))
     )
-    (property "Footprint" "" (at 46.482 99.06 90)
+    (property "Footprint" "Potentiometer_SMD:Potentiometer_Bourns_TC33X_Vertical" (at 46.482 99.06 90)
       (effects (font (size 1.27 1.27)) hide)
     )
@@
       (effects (font (size 1.27 1.27)) (justify left))
     )
-    (property "Footprint" "" (at 203.962 97.79 90)
+    (property "Footprint" "Potentiometer_SMD:Potentiometer_Bourns_TC33X_Vertical" (at 203.962 97.79 90)
       (effects (font (size 1.27 1.27)) hide)
     )
@@
       (effects (font (size 1.27 1.27)) (justify left))
     )
-    (property "Footprint" "" (at 65.532 99.06 90)
+    (property "Footprint" "Potentiometer_SMD:Potentiometer_Bourns_TC33X_Vertical" (at 65.532 99.06 90)
       (effects (font (size 1.27 1.27)) hide)
     )
@@
       (effects (font (size 1.27 1.27)) (justify left))
     )
-    (property "Footprint" "" (at 192.532 87.63 90)
+    (property "Footprint" "Resistor_SMD:R_0603_1608Metric" (at 192.532 87.63 90)
       (effects (font (size 1.27 1.27)) hide)
     )
@@
       (effects (font (size 1.27 1.27)) (justify left))
     )
-    (property "Footprint" "" (at 96.012 88.9 90)
+    (property "Footprint" "Resistor_SMD:R_0603_1608Metric" (at 96.012 88.9 90)
       (effects (font (size 1.27 1.27)) hide)
     )
@@
       (effects (font (size 1.27 1.27)) (justify left))
     )
-    (property "Footprint" "" (at 173.482 87.63 90)
+    (property "Footprint" "Resistor_SMD:R_0603_1608Metric" (at 173.482 87.63 90)
       (effects (font (size 1.27 1.27)) hide)
     )
@@
       (effects (font (size 1.27 1.27)) (justify left))
     )
-    (property "Footprint" "" (at 35.052 99.06 90)
+    (property "Footprint" "Resistor_SMD:R_0603_1608Metric" (at 35.052 99.06 90)
       (effects (font (size 1.27 1.27)) hide)
     )
@@
       (effects (font (size 1.27 1.27)) (justify left))
     )
-    (property "Footprint" "" (at 223.012 87.63 90)
+    (property "Footprint" "Resistor_SMD:R_0603_1608Metric" (at 223.012 87.63 90)
       (effects (font (size 1.27 1.27)) hide)
     )
@@
       (effects (font (size 1.27 1.27)) (justify left))
     )
-    (property "Footprint" "" (at 192.532 97.79 90)
+    (property "Footprint" "Potentiometer_SMD:Potentiometer_Bourns_TC33X_Vertical" (at 192.532 97.79 90)
       (effects (font (size 1.27 1.27)) hide)
     )
@@
       (effects (font (size 1.27 1.27)) (justify left))
     )
-    (property "Footprint" "" (at 76.962 88.9 90)
+    (property "Footprint" "Resistor_SMD:R_0603_1608Metric" (at 76.962 88.9 90)
       (effects (font (size 1.27 1.27)) hide)
     )
@@
       (effects (font (size 1.27 1.27)) (justify left))
     )
-    (property "Footprint" "" (at 223.012 97.79 90)
+    (property "Footprint" "Potentiometer_SMD:Potentiometer_Bourns_TC33X_Vertical" (at 223.012 97.79 90)
       (effects (font (size 1.27 1.27)) hide)
     )
@@
       (effects (font (size 1.27 1.27)) (justify left))
     )
-    (property "Footprint" "" (at 65.532 88.9 90)
+    (property "Footprint" "Resistor_SMD:R_0603_1608Metric" (at 65.532 88.9 90)
       (effects (font (size 1.27 1.27)) hide)
     )
@@
       (effects (font (size 1.27 1.27)) (justify left))
     )
-    (property "Footprint" "" (at 173.482 97.79 90)
+    (property "Footprint" "Potentiometer_SMD:Potentiometer_Bourns_TC33X_Vertical" (at 173.482 97.79 90)
       (effects (font (size 1.27 1.27)) hide)
     )
@@
       (effects (font (size 1.27 1.27)) (justify left))
     )
-    (property "Footprint" "" (at 203.962 87.63 90)
+    (property "Footprint" "Resistor_SMD:R_0603_1608Metric" (at 203.962 87.63 90)
       (effects (font (size 1.27 1.27)) hide)
     )
@@
       (effects (font (size 1.27 1.27)) (justify left))
     )
-    (property "Footprint" "" (at 162.052 97.79 90)
+    (property "Footprint" "Potentiometer_SMD:Potentiometer_Bourns_TC33X_Vertical" (at 162.052 97.79 90)
       (effects (font (size 1.27 1.27)) hide)
     )
@@
       (effects (font (size 1.27 1.27)) (justify left))
     )
-    (property "Footprint" "" (at 162.052 74.93 90)
+    (property "Footprint" "Resistor_SMD:R_0603_1608Metric" (at 162.052 74.93 90)
       (effects (font (size 1.27 1.27)) hide)
     )
@@
       (effects (font (size 1.27 1.27)) (justify left))
     )
-    (property "Footprint" "" (at 96.012 99.06 90)
+    (property "Footprint" "Potentiometer_SMD:Potentiometer_Bourns_TC33X_Vertical" (at 96.012 99.06 90)
       (effects (font (size 1.27 1.27)) hide)
     )
@@
       (effects (font (size 1.27 1.27)) (justify left))
     )
-    (property "Footprint" "" (at 76.962 99.06 90)
+    (property "Footprint" "Potentiometer_SMD:Potentiometer_Bourns_TC33X_Vertical" (at 76.962 99.06 90)
       (effects (font (size 1.27 1.27)) hide)
     )
@@
       (effects (font (size 1.27 1.27)) (justify left))
     )
-    (property "Footprint" "" (at 35.052 76.2 90)
+    (property "Footprint" "Resistor_SMD:R_0603_1608Metric" (at 35.052 76.2 90)
       (effects (font (size 1.27 1.27)) hide)
     )
@@
       (effects (font (size 1.27 1.27)) (justify left))
     )
-    (property "Footprint" "" (at 162.052 87.63 90)
-      (effects (font (size 1.27 1.27)) hide)
-    )
+    (property "Footprint" "Resistor_SMD:R_0603_1608Metric" (at 162.052 87.63 90)
+      (effects (font (size 1.27 1.27)) hide)
+    )

Commit message: coldent sleep so came back and did somre routing
Parts:
- removed Q10 (x2), Q11 (x2), Q7 (x2), Q8 (x2), Q9 (x2): NMOS, Package_TO_SOT_SMD:SOT-416, symbol Simulation_SPICE:NMOS
- removed R29: 10K, Resistor_SMD:R_0603_1608Metric, symbol Device:R_Trim
- added Q26 (x10): NMOS, Package_TO_SOT_SMD:SOT-416, symbol Simulation_SPICE:NMOS
- added R30: 10K, Potentiometer_SMD:Potentiometer_Bourns_TC33X_Vertical, symbol Device:R_Trim
Connections:
- net B_USB-C_BUCK_12V_SEL: now also Q26.2 (G)
- net B_USB-C_BUCK_15V_SEL: now also Q26.2 (G)
- net B_USB-C_BUCK_20V_SEL: now also Q26.2 (G)
- net B_USB-C_BUCK_5V_SEL: now also Q26.2 (G)
- net B_USB-C_BUCK_9V_SEL: now also Q26.2 (G)
- net F_USB-C_BUCK_12V_SEL: now also Q26.2 (G)
- net F_USB-C_BUCK_15V_SEL: now also Q26.2 (G)
- net F_USB-C_BUCK_20V_SEL: now also Q26.2 (G)
- net F_USB-C_BUCK_5V_SEL: now also Q26.2 (G)
- net F_USB-C_BUCK_9V_SEL: now also Q26.2 (G)
- net GND: now also Q26.3 (S), Q26.3 (S), Q26.3 (S), Q26.3 (S), Q26.3 (S), Q26.3 (S), Q26.3 (S), Q26.3 (S), Q26.3 (S), Q26.3 (S)
- net at R24.2: now also R30.1
- net at R32.2: now also Q26.1 (D) (x2)
- net at R30.2: now also Q26.1 (D) (x2)
- net at R31.2: now also Q26.1 (D) (x2)
- net at R34.2: now also Q26.1 (D) (x2)
- net at R29.2: now also Q26.1 (D)
- new net: Q26.1 (D), R30.2

Commit message: working on routing still  finnished psu section
Connections:
- net B_USB-C_BUCK_12V_SEL: now also Q26.2 (G); no longer Q26.2 (G)
- net B_USB-C_BUCK_15V_SEL: now also Q26.2 (G); no longer Q26.2 (G)
- net B_USB-C_BUCK_20V_SEL: now also Q26.2 (G); no longer Q26.2 (G)
- net B_USB-C_BUCK_5V_SEL: now also Q26.2 (G); no longer Q26.2 (G)
- net B_USB-C_BUCK_9V_SEL: now also Q26.2 (G); no longer Q26.2 (G)
- net B_USB-C_BUCK_FB: now also R24.1, R25.1, R26.1, R27.1, R28.2, R33.1; no longer R24.1, R25.1, R26.1, R27.1, R28.2, R33.1
- net B_USB-C_BUCK_OUT: now also R28.1; no longer R28.1
- net F_USB-C_BUCK_12V_SEL: now also Q26.2 (G); no longer Q26.2 (G)
- net F_USB-C_BUCK_15V_SEL: now also Q26.2 (G); no longer Q26.2 (G)
- net F_USB-C_BUCK_20V_SEL: now also Q26.2 (G); no longer Q26.2 (G)
- net F_USB-C_BUCK_5V_SEL: now also Q26.2 (G); no longer Q26.2 (G)
- net F_USB-C_BUCK_9V_SEL: now also Q26.2 (G); no longer Q26.2 (G)
- net F_USB-C_BUCK_FB: now also R24.1, R25.1, R26.1, R27.1, R28.2, R33.1; no longer R24.1, R25.1, R26.1, R27.1, R28.2, R33.1
- net F_USB-C_BUCK_OUT: now also R28.1; no longer R28.1
Changed lines of the file:
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@@
     (effects (font (size 0.75 0.75)) (justify left bottom))
   )
-  (global_label "B_USB-C_BUCK_5V_SEL" (shape input) (at 232.41 118.11 270) (fields_autoplaced)
+  (global_label "F_USB-C_BUCK_5V_SEL" (shape input) (at 232.41 118.11 270) (fields_autoplaced)
     (effects (font (size 1.27 1.27)) (justify right))
     (property "Intersheetrefs" "${INTERSHEET_REFS}" (at 232.41 143.6338 90)
@@
     )
   )
-  (global_label "B_USB-C_BUCK_9V_SEL" (shape input) (at 213.36 111.76 270) (fields_autoplaced)
+  (global_label "F_USB-C_BUCK_9V_SEL" (shape input) (at 213.36 111.76 270) (fields_autoplaced)
     (effects (font (size 1.27 1.27)) (justify right))
     (property "Intersheetrefs" "${INTERSHEET_REFS}" (at 213.36 137.2838 90)
@@
     )
   )
-  (global_label "B_USB-C_BUCK_12V_SEL" (shape input) (at 201.93 118.11 270) (fields_autoplaced)
+  (global_label "F_USB-C_BUCK_12V_SEL" (shape input) (at 201.93 118.11 270) (fields_autoplaced)
     (effects (font (size 1.27 1.27)) (justify right))
     (property "Intersheetrefs" "${INTERSHEET_REFS}" (at 201.93 144.8433 90)
@@
     )
   )
-  (global_label "B_USB-C_BUCK_OUT" (shape input) (at 163.83 71.12 90) (fields_autoplaced)
+  (global_label "F_USB-C_BUCK_OUT" (shape input) (at 163.83 71.12 90) (fields_autoplaced)
     (effects (font (size 1.27 1.27)) (justify left))
     (property "Intersheetrefs" "${INTERSHEET_REFS}" (at 163.83 48.6199 90)
@@
     )
   )
-  (global_label "F_USB-C_BUCK_9V_SEL" (shape input) (at 86.36 113.03 270) (fields_autoplaced)
+  (global_label "B_USB-C_BUCK_9V_SEL" (shape input) (at 86.36 113.03 270) (fields_autoplaced)
     (effects (font (size 1.27 1.27)) (justify right))
     (property "Intersheetrefs" "${INTERSHEET_REFS}" (at 86.36 138.3724 90)
@@
     )
   )
-  (global_label "B_USB-C_BUCK_20V_SEL" (shape input) (at 171.45 118.11 270) (fields_autoplaced)
+  (global_label "F_USB-C_BUCK_20V_SEL" (shape input) (at 171.45 118.11 270) (fields_autoplaced)
     (effects (font (size 1.27 1.27)) (justify right))
     (property "Intersheetrefs" "${INTERSHEET_REFS}" (at 171.45 144.8433 90)
@@
     )
   )
-  (global_label "F_USB-C_BUCK_OUT" (shape input) (at 36.83 72.39 90) (fields_autoplaced)
+  (global_label "B_USB-C_BUCK_OUT" (shape input) (at 36.83 72.39 90) (fields_autoplaced)
     (effects (font (size 1.27 1.27)) (justify left))
     (property "Intersheetrefs" "${INTERSHEET_REFS}" (at 36.83 50.0713 90)
@@
     )
   )
-  (global_label "F_USB-C_BUCK_15V_SEL" (shape input) (at 55.88 113.03 270) (fields_autoplaced)
+  (global_label "B_USB-C_BUCK_15V_SEL" (shape input) (at 55.88 113.03 270) (fields_autoplaced)
     (effects (font (size 1.27 1.27)) (justify right))
     (property "Intersheetrefs" "${INTERSHEET_REFS}" (at 55.88 139.5819 90)
@@
     )
   )
-  (global_label "F_USB-C_BUCK_FB" (shape input) (at 97.79 82.55 0) (fields_autoplaced)
+  (global_label "B_USB-C_BUCK_FB" (shape input) (at 97.79 82.55 0) (fields_autoplaced)
     (effects (font (size 1.27 1.27)) (justify left))
     (property "Intersheetrefs" "${INTERSHEET_REFS}" (at 118.8387 82.55 0)
@@
     )
   )
-  (global_label "B_USB-C_BUCK_FB" (shape input) (at 224.79 81.28 0) (fields_autoplaced)
+  (global_label "F_USB-C_BUCK_FB" (shape input) (at 224.79 81.28 0) (fields_autoplaced)
     (effects (font (size 1.27 1.27)) (justify left))
     (property "Intersheetrefs" "${INTERSHEET_REFS}" (at 246.0201 81.28 0)
@@
     )
   )
-  (global_label "F_USB-C_BUCK_5V_SEL" (shape input) (at 105.41 119.38 270) (fields_autoplaced)
+  (global_label "B_USB-C_BUCK_5V_SEL" (shape input) (at 105.41 119.38 270) (fields_autoplaced)
     (effects (font (size 1.27 1.27)) (justify right))
     (property "Intersheetrefs" "${INTERSHEET_REFS}" (at 105.41 144.7224 90)
@@
     )
   )
-  (global_label "F_USB-C_BUCK_12V_SEL" (shape input) (at 74.93 119.38 270) (fields_autoplaced)
+  (global_label "B_USB-C_BUCK_12V_SEL" (shape input) (at 74.93 119.38 270) (fields_autoplaced)
     (effects (font (size 1.27 1.27)) (justify right))
     (property "Intersheetrefs" "${INTERSHEET_REFS}" (at 74.93 145.9319 90)
@@
     )
   )
-  (global_label "F_USB-C_BUCK_20V_SEL" (shape input) (at 44.45 119.38 270) (fields_autoplaced)
+  (global_label "B_USB-C_BUCK_20V_SEL" (shape input) (at 44.45 119.38 270) (fields_autoplaced)
     (effects (font (size 1.27 1.27)) (justify right))
     (property "Intersheetrefs" "${INTERSHEET_REFS}" (at 44.45 145.9319 90)
@@
     )
   )
-  (global_label "B_USB-C_BUCK_15V_SEL" (shape input) (at 182.88 111.76 270) (fields_autoplaced)
+  (global_label "F_USB-C_BUCK_15V_SEL" (shape input) (at 182.88 111.76 270) (fields_autoplaced)
     (effects (font (size 1.27 1.27)) (justify right))
     (property "Intersheetrefs" "${INTERSHEET_REFS}" (at 182.88 138.4933 90)

Commit message: finaliseing pcb layout will come back later for a fresh look
Other:
- company: (none) -> MICK MAKE
- title: (none) -> 200W USB PD 3.1 HUB
Changed lines of the file:
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@@
 (kicad_sch (version 20230121) (generator eeschema)
   (paper "A4")
+  (title_block
+    (title "200W USB PD 3.1 HUB")
+    (date "2023-10-03")
+    (rev "A")
+    (company "MICK MAKE")
+    (comment 1 "THIS IS A 2X 100W USB PD SOURCE ")
+    (comment 2 "HUB USB SPEC 3.1")
+    (comment 3 "TOTAL SYSTEM POWER IS ~275w")
+  )
   (junction (at 194.31 148.59) (diameter 0) (color 0 0 0 0)
   )

Commit message: fixed DP issues and finneshed overall routeing
Parts:
- renumbered Q26 to Q10, Q26 to Q11, Q26 to Q12, Q26 to Q13, Q26 to Q14, Q26 to Q15, Q26 to Q16, Q26 to Q7, Q26 to Q8, Q26 to Q9, R24 to R29, R25 to R31, R30 to R32, R26 to R33, R31 to R34, R27 to R35, R32 to R36, R33 to R37, R34 to R38, R28 to R39, R24 to R40, R29 to R41, R25 to R42, R30 to R43, R26 to R44, R31 to R45, R27 to R46, R32 to R47, R33 to R48, R34 to R49

Commit message: minor revisions
Parts:
- Q10, Q11, Q12, Q13, Q14, Q15, Q16, Q7, Q8, Q9: value NMOS -> NTA7002NT1G
Changed lines of the file:
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@@
       (effects (font (size 1.27 1.27)) (justify left))
     )
-    (property "Value" "NMOS" (at 34.163 119.3873 0)
+    (property "Value" "NTA7002NT1G" (at 34.163 119.3873 0)
       (effects (font (size 1.27 1.27)) (justify left))
     )
@@
       (effects (font (size 1.27 1.27)) (justify left))
     )
-    (property "Value" "NMOS" (at 161.163 118.1173 0)
+    (property "Value" "NTA7002NT1G" (at 161.163 118.1173 0)
       (effects (font (size 1.27 1.27)) (justify left))
     )
@@
       (effects (font (size 1.27 1.27)) (justify left))
     )
-    (property "Value" "NMOS" (at 203.073 111.7673 0)
+    (property "Value" "NTA7002NT1G" (at 203.073 111.7673 0)
       (effects (font (size 1.27 1.27)) (justify left))
     )
@@
       (effects (font (size 1.27 1.27)) (justify left))
     )
-    (property "Value" "NMOS" (at 76.073 113.0373 0)
+    (property "Value" "NTA7002NT1G" (at 76.073 113.0373 0)
       (effects (font (size 1.27 1.27)) (justify left))
     )
@@
       (effects (font (size 1.27 1.27)) (justify left))
     )
-    (property "Value" "NMOS" (at 45.593 113.0373 0)
+    (property "Value" "NTA7002NT1G" (at 45.593 113.0373 0)
       (effects (font (size 1.27 1.27)) (justify left))
     )
@@
       (effects (font (size 1.27 1.27)) (justify left))
     )
-    (property "Value" "NMOS" (at 191.643 118.1173 0)
+    (property "Value" "NTA7002NT1G" (at 191.643 118.1173 0)
       (effects (font (size 1.27 1.27)) (justify left))
     )
@@
       (effects (font (size 1.27 1.27)) (justify left))
     )
-    (property "Value" "NMOS" (at 172.593 111.7673 0)
+    (property "Value" "NTA7002NT1G" (at 172.593 111.7673 0)
       (effects (font (size 1.27 1.27)) (justify left))
     )
@@
       (effects (font (size 1.27 1.27)) (justify left))
     )
-    (property "Value" "NMOS" (at 95.123 119.3873 0)
+    (property "Value" "NTA7002NT1G" (at 95.123 119.3873 0)
       (effects (font (size 1.27 1.27)) (justify left))
     )
@@
       (effects (font (size 1.27 1.27)) (justify left))
     )
-    (property "Value" "NMOS" (at 64.643 119.3873 0)
+    (property "Value" "NTA7002NT1G" (at 64.643 119.3873 0)
       (effects (font (size 1.27 1.27)) (justify left))
     )
@@
       (effects (font (size 1.27 1.27)) (justify left))
     )
-    (property "Value" "NMOS" (at 222.123 118.1173 0)
-      (effects (font (size 1.27 1.27)) (justify left))
-    )
+    (property "Value" "NTA7002NT1G" (at 222.123 118.1173 0)
+      (effects (font (size 1.27 1.27)) (justify left))
+    )
