File: hardware/FRONT_PANNEL_DISPLAY.kicad_sch (KiCad schematic)
At the start: 17 parts, among them SW1 SW_Push, SW2 SW_Push, U7 AS1115-BSST, U9 LTC-5723HR

Commit message: working on hardware
Parts:
- added D30: 10W, Diode_SMD:D_0603_1608Metric, symbol Device:LED
- added D31: 20W, Diode_SMD:D_0603_1608Metric, symbol Device:LED
- added D32: 40W, Diode_SMD:D_0603_1608Metric, symbol Device:LED
- added D33: 65W, Diode_SMD:D_0603_1608Metric, symbol Device:LED
- added D34: 100W, Diode_SMD:D_0603_1608Metric, symbol Device:LED
- added R103: 10K, symbol Device:R
- added SW3: SW_Push, symbol Switch:SW_Push
- C110: renamed from C93; footprint (none) -> Capacitor_SMD:C_0603_1608Metric
- C111: renamed from C92; footprint (none) -> Capacitor_SMD:C_0603_1608Metric
- D23, D24, D25, D26, D27, D28, D29: footprint (none) -> Diode_SMD:D_0603_1608Metric
- renumbered R99 to R100, R102 to R101, R101 to R102, R98 to R99
Connections:
- net +3V3: now also R103.1
- net DISP_SEG_A: now also D30.2 (A)
- net DISP_SEG_B: now also D31.2 (A)
- net DISP_SEG_C: now also D32.2 (A)
- net DISP_SEG_D: now also D33.2 (A)
- net DISP_SEG_E: now also D34.2 (A)
- net GND: now also SW3.2
- net DISP_DIG_6: now reaches U7.9 (DIG6)
- net DISP_DIG_6: now also D30.1 (K), D31.1 (K), D32.1 (K), D33.1 (K), D34.1 (K)
- new net MODE_BTN: R103.2, SW3.1
Other:
- note added: "DISPLAY DRIVER"
- note added: "FRONT DISPLAY"
- note added: "INFO LEDS"
- note added: "USER INPUT"
- moved on the sheet: C110, C111, D23, D24, D25, D26, D27, D28, D29, R100, R101, R102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

Commit message: working assighning footprints still
Parts:
- R100, R101, R102, R103, R99: footprint (none) -> Resistor_SMD:R_0603_1608Metric
Changed lines of the file:
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@@
       (effects (font (size 1.27 1.27)) (justify left))
     )
-    (property "Footprint" "" (at 59.182 124.46 90)
+    (property "Footprint" "Resistor_SMD:R_0603_1608Metric" (at 59.182 124.46 90)
       (effects (font (size 1.27 1.27)) hide)
     )
@@
       (effects (font (size 1.27 1.27)) (justify left))
     )
-    (property "Footprint" "" (at 60.452 180.34 90)
+    (property "Footprint" "Resistor_SMD:R_0603_1608Metric" (at 60.452 180.34 90)
       (effects (font (size 1.27 1.27)) hide)
     )
@@
       (effects (font (size 1.27 1.27)) (justify left))
     )
-    (property "Footprint" "" (at 59.182 153.67 90)
+    (property "Footprint" "Resistor_SMD:R_0603_1608Metric" (at 59.182 153.67 90)
       (effects (font (size 1.27 1.27)) hide)
     )
@@
       (effects (font (size 1.27 1.27)) (justify left))
     )
-    (property "Footprint" "" (at 51.562 39.37 90)
+    (property "Footprint" "Resistor_SMD:R_0603_1608Metric" (at 51.562 39.37 90)
       (effects (font (size 1.27 1.27)) hide)
     )
@@
       (effects (font (size 1.27 1.27)) (justify left))
     )
-    (property "Footprint" "" (at 43.942 39.37 90)
-      (effects (font (size 1.27 1.27)) hide)
-    )
+    (property "Footprint" "Resistor_SMD:R_0603_1608Metric" (at 43.942 39.37 90)
+      (effects (font (size 1.27 1.27)) hide)
+    )

Commit message: FINALY starting the pcb
Parts:
- SW1, SW2, SW3: footprint (none) -> Button_Switch_THT:SW_PUSH_6mm
Changed lines of the file:
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@@
       (effects (font (size 1.27 1.27)))
     )
-    (property "Footprint" "" (at 73.66 182.88 0)
+    (property "Footprint" "Button_Switch_THT:SW_PUSH_6mm" (at 73.66 182.88 0)
       (effects (font (size 1.27 1.27)) hide)
     )
@@
       (effects (font (size 1.27 1.27)))
     )
-    (property "Footprint" "" (at 72.39 127 0)
+    (property "Footprint" "Button_Switch_THT:SW_PUSH_6mm" (at 72.39 127 0)
       (effects (font (size 1.27 1.27)) hide)
     )
@@
       (effects (font (size 1.27 1.27)))
     )
-    (property "Footprint" "" (at 72.39 156.21 0)
-      (effects (font (size 1.27 1.27)) hide)
-    )
+    (property "Footprint" "Button_Switch_THT:SW_PUSH_6mm" (at 72.39 156.21 0)
+      (effects (font (size 1.27 1.27)) hide)
+    )

Commit message: finaliseing pcb layout will come back later for a fresh look
Other:
- company: (none) -> MICK MAKE
- title: (none) -> 200W USB PD 3.1 HUB
Changed lines of the file:
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@@
 (kicad_sch (version 20230121) (generator eeschema)
   (paper "A4")
+  (title_block
+    (title "200W USB PD 3.1 HUB")
+    (date "2023-10-03")
+    (rev "A")
+    (company "MICK MAKE")
+    (comment 1 "THIS IS A 2X 100W USB PD SOURCE ")
+    (comment 2 "HUB USB SPEC 3.1")
+    (comment 3 "TOTAL SYSTEM POWER IS ~275w")
+  )
   (junction (at 261.62 99.06) (diameter 0) (color 0 0 0 0)
   )

Commit message: switched can tranceiver to combo controler and tranceiver
Parts:
- added TP31, TP32, TP33: TestPoint, TestPoint:TestPoint_Pad_D1.0mm, symbol Connector:TestPoint
Connections:
- net at U7.12 (KEYB): now also TP33.1
- net at U7.7 (DIG4): now also TP31.1
- net at U7.8 (DIG5): now also TP32.1
Changed lines of the file:
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@@
 	(wire
 		(pts
+			(xy 92.71 73.66) (xy 107.95 73.66)
+		)
+		(stroke
+			(width 0)
+			(type default)
+		)
+	)
+	(wire
+		(pts
 			(xy 35.56 44.45) (xy 35.56 43.18)
 		)
@@
 		)
 	)
+	(wire
+		(pts
+			(xy 92.71 76.2) (xy 107.95 76.2)
+		)
+		(stroke
+			(width 0)
+			(type default)
+		)
+	)
 	(polyline
 		(pts
@@
 	(wire
 		(pts
+			(xy 92.71 88.9) (xy 95.25 88.9)
+		)
+		(stroke
+			(width 0)
+			(type default)
+		)
+	)
+	(wire
+		(pts
 			(xy 204.47 99.06) (xy 204.47 106.68)
 		)
@@
 	(wire
 		(pts
-			(xy 118.11 86.36) (xy 118.11 53.34)
+			(xy 120.65 86.36) (xy 120.65 53.34)
 		)
 		(stroke
@@
 	(wire
 		(pts
-			(xy 92.71 86.36) (xy 118.11 86.36)
+			(xy 92.71 86.36) (xy 120.65 86.36)
 		)
 		(stroke
@@
 	(wire
 		(pts
-			(xy 118.11 53.34) (xy 92.71 53.34)
+			(xy 92.71 53.34) (xy 120.65 53.34)
 		)
 		(stroke
@@
 	(global_label "DISP_SEG_G"
 		(shape input)
-		(at 118.11 53.34 0)
+		(at 120.65 53.34 0)
 		(fields_autoplaced yes)
 		(effects
@@
 		)
 		(property "Intersheetrefs" "${INTERSHEET_REFS}"
-			(at 132.2038 53.34 0)
+			(at 134.7438 53.34 0)
 			(effects
 				(font
@@
 	)
 	(symbol
+		(lib_id "Connector:TestPoint")
+		(at 107.95 76.2 180)
+		(unit 1)
+		(exclude_from_sim no)
+		(in_bom yes)
+		(on_board yes)
+		(dnp no)
+		(fields_autoplaced yes)
+		(property "Reference" "TP32"
+			(at 109.347 78.2898 0)
+			(effects
+				(font
+					(size 1.27 1.27)
+				)
+				(justify right)
+			)
+		)
+		(property "Value" "TestPoint"
+			(at 109.347 80.7141 0)
+			(effects
+				(font
+					(size 1.27 1.27)
+				)
+				(justify right)
+			)
+		)
+		(property "Footprint" "TestPoint:TestPoint_Pad_D1.0mm"
+			(at 102.87 76.2 0)
+			(effects
+				(font
+					(size 1.27 1.27)
+				)
+				(hide yes)
+			)
+		)
+		(property "Datasheet" "~"
+			(at 102.87 76.2 0)
+			(effects
+				(font
+					(size 1.27 1.27)
+				)
+				(hide yes)
+			)
+		)
+		(property "Description" "test point"
+			(at 107.95 76.2 0)
+			(effects
+				(font
+					(size 1.27 1.27)
+				)
+				(hide yes)
+			)
+		)
+		(pin "1"
+		)
+		(instances
+			(project "usbc-car-module"
+				(path "/fae025e9-99c5-40c1-af6f-99dc1edbfa43/ba7fd60c-2f9a-4947-88c0-3b779b991f83"
+					(reference "TP32")
+					(unit 1)
+				)
+			)
+		)
+	)
+	(symbol
 		(lib_id "Device:LED")
 		(at 187.96 83.82 180)
@@
 	)
 	(symbol
+		(lib_id "Connector:TestPoint")
+		(at 107.95 73.66 0)
+		(unit 1)
+		(exclude_from_sim no)
+		(in_bom yes)
+		(on_board yes)
+		(dnp no)
+		(fields_autoplaced yes)
+		(property "Reference" "TP31"
+			(at 109.347 69.1458 0)
+			(effects
+				(font
+					(size 1.27 1.27)
+				)
+				(justify left)
+			)
+		)
+		(property "Value" "TestPoint"
+			(at 109.347 71.5701 0)
+			(effects
+				(font
+					(size 1.27 1.27)
+				)
+				(justify left)
+			)
+		)
+		(property "Footprint" "TestPoint:TestPoint_Pad_D1.0mm"
+			(at 113.03 73.66 0)
+			(effects
+				(font
+					(size 1.27 1.27)
+				)
+				(hide yes)
+			)
+		)
+		(property "Datasheet" "~"
+			(at 113.03 73.66 0)
+			(effects
+				(font
+					(size 1.27 1.27)
+				)
+				(hide yes)
+			)
+		)
+		(property "Description" "test point"
+			(at 107.95 73.66 0)
+			(effects
+				(font
+					(size 1.27 1.27)
+				)
+				(hide yes)
+			)
+		)
+		(pin "1"
+		)
+		(instances
+			(project "usbc-car-module"
+				(path "/fae025e9-99c5-40c1-af6f-99dc1edbfa43/ba7fd60c-2f9a-4947-88c0-3b779b991f83"
+					(reference "TP31")
+					(unit 1)
+				)
+			)
+		)
+	)
+	(symbol
 		(lib_id "Switch:SW_Push")
 		(at 72.39 161.29 0)
@@
 					(unit 1)
 				)
+			)
+		)
+	)
+	(symbol
+		(lib_id "Connector:TestPoint")
+		(at 95.25 88.9 180)
+		(unit 1)
+		(exclude_from_sim no)
+		(in_bom yes)
+		(on_board yes)
+		(dnp no)
+		(fields_autoplaced yes)
+		(property "Reference" "TP33"
+			(at 96.647 90.9898 0)
+			(effects
+				(font
+					(size 1.27 1.27)
+				)
+				(justify right)
+			)
+		)
+		(property "Value" "TestPoint"
+			(at 96.647 93.4141 0)
+			(effects
+				(font
+					(size 1.27 1.27)
+				)
+				(justify right)
+			)
+		)
+		(property "Footprint" "TestPoint:TestPoint_Pad_D1.0mm"
+			(at 90.17 88.9 0)
+			(effects
+				(font
+					(size 1.27 1.27)
+				)
+				(hide yes)
+			)
+		)
+		(property "Datasheet" "~"
+			(at 90.17 88.9 0)
+			(effects
+				(font
+					(size 1.27 1.27)
+				)
+				(hide yes)
+			)
+		)
+		(property "Description" "test point"
+			(at 95.25 88.9 0)
+			(effects
+				(font
+					(size 1.27 1.27)
+				)
+				(hide yes)
+			)
+		)
+		(pin "1"
+		)
+		(instances
+			(project "usbc-car-module"
+				(path "/fae025e9-99c5-40c1-af6f-99dc1edbfa43/ba7fd60c-2f9a-4947-88c0-3b779b991f83"
+					(reference "TP33")
+					(unit 1)
+				)

Commit message: migrated to the esp32-s2 and starting new board revison
Parts:
- renumbered C110 to C129, C111 to C130, D23 to D19, D30 to D20, D24 to D21, D31 to D22, D25 to D23, D32 to D24, D26 to D25, D33 to D26, D34 to D28, D28 to D29, D29 to D30, R99 to R103, R100 to R104, R101 to R105, R102 to R106, R103 to R107, TP31 to TP47, TP32 to TP48, TP33 to TP49, U9 to U13, U7 to U14
